File: laserctrl/psu.sch (KiCad schematic (older format))
At the start: 23 parts, among them IC3 TPS78233, U2 MC34063

Commit message: Deleted the A-axis, it's getting too cramped with limited 328 I/O
Parts:
- renumbered C22 to C10, C23 to C11, C9 to C4, C15 to C5, C18 to C6, C19 to C7, C20 to C8, C50 to C9, D3 to D1, L2 to L1, R27 to R5, R31 to R6, R32 to R7, U2 to U1
Changed lines of the file:
@@
-EESchema Schematic File Version 2  date 2011-10-22T12:24:09 CEST
+EESchema Schematic File Version 2  date 2011-10-22T21:04:28 CEST
 LIBS:power
 LIBS:device
@@
 EELAYER END
 $Descr A4 11700 8267
-Sheet 6 6
+Sheet 6 5
 Title ""
 Date "22 oct 2011"
@@
 	6650 3900 6650 3950
 $Comp
-L GND #PWR23
+L GND #PWR24
 U 1 1 4EA1CE90
 P 4300 7100
-F 0 "#PWR23" H 4300 7100 30  0001 C CNN
+F 0 "#PWR24" H 4300 7100 30  0001 C CNN
 F 1 "GND" H 4300 7030 30  0001 C CNN
 	1    4300 7100
@@
 $EndComp
 $Comp
-L GND #PWR22
+L GND #PWR23
 U 1 1 4EA1CE88
 P 3900 7100
-F 0 "#PWR22" H 3900 7100 30  0001 C CNN
+F 0 "#PWR23" H 3900 7100 30  0001 C CNN
 F 1 "GND" H 3900 7030 30  0001 C CNN
 	1    3900 7100
@@
 $EndComp
 $Comp
-L GND #PWR20
+L GND #PWR21
 U 1 1 4EA1CE84
 P 3500 7100
-F 0 "#PWR20" H 3500 7100 30  0001 C CNN
+F 0 "#PWR21" H 3500 7100 30  0001 C CNN
 F 1 "GND" H 3500 7030 30  0001 C CNN
 	1    3500 7100
@@
 $EndComp
 $Comp
-L GND #PWR29
+L GND #PWR30
 U 1 1 4EA1CE05
 P 6350 4400
-F 0 "#PWR29" H 6350 4400 30  0001 C CNN
+F 0 "#PWR30" H 6350 4400 30  0001 C CNN
 F 1 "GND" H 6350 4330 30  0001 C CNN
 	1    6350 4400
@@
 $EndComp
 $Comp
-L C C50
+L C C9
 U 1 1 4EA1CDFC
 P 6350 4150
-F 0 "C50" H 6400 4250 50  0000 L CNN
+F 0 "C9" H 6400 4250 50  0000 L CNN
 F 1 "1uF" H 6400 4050 50  0000 L CNN
 	1    6350 4150
@@
 $EndComp
 $Comp
-L +3.3V #PWR28
+L +3.3V #PWR29
 U 1 1 4EA1CDEC
 P 6350 3750
-F 0 "#PWR28" H 6350 3710 30  0001 C CNN
+F 0 "#PWR29" H 6350 3710 30  0001 C CNN
 F 1 "+3.3V" H 6350 3860 30  0000 C CNN
 	1    6350 3750
@@
 $EndComp
 $Comp
-L GND #PWR25
+L GND #PWR26
 U 1 1 4EA1CDD6
 P 5500 4600
-F 0 "#PWR25" H 5500 4600 30  0001 C CNN
+F 0 "#PWR26" H 5500 4600 30  0001 C CNN
 F 1 "GND" H 5500 4530 30  0001 C CNN
 	1    5500 4600
@@
 $EndComp
 $Comp
-L +5V #PWR24
+L +5V #PWR25
 U 1 1 4EA1CDCB
 P 4800 3800
-F 0 "#PWR24" H 4800 3890 20  0001 C CNN
+F 0 "#PWR25" H 4800 3890 20  0001 C CNN
 F 1 "+5V" H 4800 3890 30  0000 C CNN
 	1    4800 3800
@@
 $EndComp
 $Comp
-L GND #PWR19
+L GND #PWR20
 U 1 1 4D879ADC
 P 3100 7100
-F 0 "#PWR19" H 3100 7100 30  0001 C CNN
+F 0 "#PWR20" H 3100 7100 30  0001 C CNN
 F 1 "GND" H 3100 7030 30  0001 C CNN
 	1    3100 7100
@@
 3mm mounting holes at the corners of the board and heatsink
 $Comp
-L GND #PWR16
+L GND #PWR17
 U 1 1 4D87999F
 P 2700 7100
-F 0 "#PWR16" H 2700 7100 30  0001 C CNN
+F 0 "#PWR17" H 2700 7100 30  0001 C CNN
 F 1 "GND" H 2700 7030 30  0001 C CNN
 	1    2700 7100
@@
 $EndComp
 $Comp
-L GND #PWR15
+L GND #PWR16
 U 1 1 4D87999A
 P 2300 7100
-F 0 "#PWR15" H 2300 7100 30  0001 C CNN
+F 0 "#PWR16" H 2300 7100 30  0001 C CNN
 F 1 "GND" H 2300 7030 30  0001 C CNN
 	1    2300 7100
@@
 $EndComp
 $Comp
-L GND #PWR13
+L GND #PWR14
 U 1 1 4D879997
 P 1900 7100
-F 0 "#PWR13" H 1900 7100 30  0001 C CNN
+F 0 "#PWR14" H 1900 7100 30  0001 C CNN
 F 1 "GND" H 1900 7030 30  0001 C CNN
 	1    1900 7100
@@
 $EndComp
 $Comp
-L GND #PWR12
+L GND #PWR13
 U 1 1 4D879990
 P 1500 7100
-F 0 "#PWR12" H 1500 7100 30  0001 C CNN
+F 0 "#PWR13" H 1500 7100 30  0001 C CNN
 F 1 "GND" H 1500 7030 30  0001 C CNN
 	1    1500 7100
@@
 Distributed decoupling caps
 $Comp
-L +5V #PWR26
+L +5V #PWR27
 U 1 1 4D0BB423
 P 5850 2200
-F 0 "#PWR26" H 5850 2290 20  0001 C CNN
+F 0 "#PWR27" H 5850 2290 20  0001 C CNN
 F 1 "+5V" H 5850 2290 30  0000 C CNN
 	1    5850 2200
@@
 $EndComp
 $Comp
-L GND #PWR27
+L GND #PWR28
 U 1 1 4D04D42D
 P 5850 3150
-F 0 "#PWR27" H 5850 3150 30  0001 C CNN
+F 0 "#PWR28" H 5850 3150 30  0001 C CNN
 F 1 "GND" H 5850 3080 30  0001 C CNN
 	1    5850 3150
@@
 $EndComp
 $Comp
-L C C23
+L C C11
 U 1 1 4D04D398
 P 6650 4150
-F 0 "C23" H 6700 4250 50  0000 L CNN
+F 0 "C11" H 6700 4250 50  0000 L CNN
 F 1 "100nF" H 6700 4050 50  0000 L CNN
 	1    6650 4150
@@
 $EndComp
 $Comp
-L C C22
+L C C10
 U 1 1 4D04D394
 P 6550 2800
-F 0 "C22" H 6600 2900 50  0000 L CNN
+F 0 "C10" H 6600 2900 50  0000 L CNN
 F 1 "100nF" H 6500 2550 50  0000 L CNN
 	1    6550 2800
@@
 $EndComp
 $Comp
-L C C20
+L C C8
 U 1 1 4D04D38C
 P 6300 2800
-F 0 "C20" H 6350 2900 50  0000 L CNN
+F 0 "C8" H 6350 2900 50  0000 L CNN
 F 1 "100nF" H 6250 2550 50  0000 L CNN
 	1    6300 2800
@@
 $EndComp
 $Comp
-L C C19
+L C C7
 U 1 1 4D04D33D
 P 6050 2800
-F 0 "C19" H 6100 2900 50  0000 L CNN
+F 0 "C7" H 6100 2900 50  0000 L CNN
 F 1 "100nF" H 6000 2550 50  0000 L CNN
 	1    6050 2800
@@
 $EndComp
 $Comp
-L C C18
+L C C6
 U 1 1 4D04D22A
 P 5350 2800
-F 0 "C18" H 5400 2900 50  0000 L CNN
+F 0 "C6" H 5400 2900 50  0000 L CNN
 F 1 "10uF" H 5400 2700 50  0000 L CNN
 	1    5350 2800
@@
 $EndComp
 $Comp
-L CAPAPOL C15
+L CAPAPOL C5
 U 1 1 4D04D0AE
 P 5050 2800
-F 0 "C15" H 5100 2900 50  0000 L CNN
+F 0 "C5" H 5100 2900 50  0000 L CNN
 F 1 "220uF" H 5100 2700 50  0000 L CNN
 	1    5050 2800
@@
 $EndComp
 $Comp
-L INDUCTOR L2
+L INDUCTOR L1
 U 1 1 4D04CFE3
 P 4650 2600
-F 0 "L2" V 4600 2600 40  0000 C CNN
+F 0 "L1" V 4600 2600 40  0000 C CNN
 F 1 "330uH" V 4750 2600 40  0000 C CNN
 	1    4650 2600
@@
 $EndComp
 $Comp
-L DIODESCH D3
+L DIODESCH D1
 U 1 1 4D04CF74
 P 4250 2800
-F 0 "D3" H 4250 2900 40  0000 C CNN
+F 0 "D1" H 4250 2900 40  0000 C CNN
 F 1 "SK 54" H 4250 2700 40  0000 C CNN
 	1    4250 2800
@@
 $EndComp
 $Comp
-L C C9
+L C C4
 U 1 1 4D04CF13
 P 2200 3100
-F 0 "C9" H 2250 3200 50  0000 L CNN
+F 0 "C4" H 2250 3200 50  0000 L CNN
 F 1 "82pF" H 2250 3000 50  0000 L CNN
 	1    2200 3100
@@
 $EndComp
 $Comp
-L GND #PWR14
+L GND #PWR15
 U 1 1 4D04CF0D
 P 2200 3450
-F 0 "#PWR14" H 2200 3450 30  0001 C CNN
+F 0 "#PWR15" H 2200 3450 30  0001 C CNN
 F 1 "GND" H 2200 3380 30  0001 C CNN
 	1    2200 3450
@@
 $EndComp
 $Comp
-L GND #PWR21
+L GND #PWR22
 U 1 1 4D04CF06
 P 3900 3450
-F 0 "#PWR21" H 3900 3450 30  0001 C CNN
+F 0 "#PWR22" H 3900 3450 30  0001 C CNN
 F 1 "GND" H 3900 3380 30  0001 C CNN
 	1    3900 3450
@@
 $EndComp
 $Comp
-L GND #PWR18
+L GND #PWR19
 U 1 1 4D04CF02
 P 3050 3150
-F 0 "#PWR18" H 3050 3150 30  0001 C CNN
+F 0 "#PWR19" H 3050 3150 30  0001 C CNN
 F 1 "GND" H 3050 3080 30  0001 C CNN
 	1    3050 3150
@@
 $EndComp
 $Comp
-L R R32
+L R R7
 U 1 1 4D04CED4
 P 4350 2300
-F 0 "R32" V 4430 2300 50  0000 C CNN
+F 0 "R7" V 4430 2300 50  0000 C CNN
 F 1 "3k" V 4350 2300 50  0000 C CNN
 	1    4350 2300
@@
 $EndComp
 $Comp
-L R R31
+L R R6
 U 1 1 4D04CEB9
 P 3900 3100
-F 0 "R31" V 3980 3100 50  0000 C CNN
+F 0 "R6" V 3980 3100 50  0000 C CNN
 F 1 "1k" V 3900 3100 50  0000 C CNN
 	1    3900 3100
@@
 $EndComp
 $Comp
-L R R27
+L R R5
 U 1 1 4D04CE98
 P 2650 2000
-F 0 "R27" V 2730 2000 50  0000 C CNN
+F 0 "R5" V 2730 2000 50  0000 C CNN
 F 1 "0.22R" V 2650 2000 50  0000 C CNN
 	1    2650 2000
@@
 $EndComp
 $Comp
-L +24V #PWR17
+L +24V #PWR18
 U 1 1 4D04CE42
 P 3050 1950
-F 0 "#PWR17" H 3050 1900 20  0001 C CNN
+F 0 "#PWR18" H 3050 1900 20  0001 C CNN
 F 1 "+24V" H 3050 2050 30  0000 C CNN
 	1    3050 1950
@@
 $EndComp
 $Comp
-L MC34063 U2
+L MC34063 U1
 U 1 1 4D04CE01
 P 3050 2550
-F 0 "U2" H 3200 2900 60  0000 L CNN
+F 0 "U1" H 3200 2900 60  0000 L CNN
 F 1 "MC34063" H 3150 2200 60  0000 L CNN
 	1    3050 2550

Commit message: Started work on ARM 32
Parts:
- removed C11: 100nF, symbol C
- removed C9: 1uF, symbol C
- removed IC3: TPS78233, symbol TPS78233
- added C? (x3): 10nF, symbol C
- added C? (x3): 100nF, symbol C
- added D? (x2): DIODE, symbol DIODE
- added FB?: FILTER, symbol FILTER
- added P?: CONN_2, symbol CONN_2
- C8: value 100nF -> 10nF
- R6: value 1k -> 11k
- R7: value 3k -> 18k
Connections:
- net labels added: +3.3VADC, +BATT
- net labels removed: +5V
- wire segments 59 -> 44
