File: laserctrl/psu.sch (KiCad schematic (older format))
At the start: 35 parts, among them P24 battery, P27 Power, U7 MC34063, U8 MC78L05ABDG

Commit message: Generated the BOM and figured out what parts to buy at ELFA and Mouser
Parts:
- C87: value 4.7uF/6.3 -> 4.7uF/6.3V
Changed lines of the file:
@@
-EESchema Schematic File Version 2  date 2011-11-28T22:17:03 CET
+EESchema Schematic File Version 2  date 2011-12-03T21:12:32 CET
 LIBS:power
 LIBS:device
@@
 Sheet 10 10
 Title ""
-Date "27 nov 2011"
+Date "3 dec 2011"
 Rev ""
 Comp ""
@@
 P 3050 4950
 F 0 "C87" H 3100 5050 50  0000 L CNN
-F 1 "4.7uF/6.3" H 3100 4850 50  0000 L CNN
+F 1 "4.7uF/6.3V" H 3100 4850 50  0000 L CNN
 	1    3050 4950
 	1    0    0    -1

Commit message: Did some more rev2 schematic changes
Parts:
- removed P27: Power, symbol CONN_2
Connections:
- wire segments 71 -> 67
Changed lines of the file:
@@
-EESchema Schematic File Version 2  date Sat 13 Oct 2012 04:06:36 PM CEST
+EESchema Schematic File Version 2  date Sun 14 Oct 2012 04:23:31 PM CEST
 LIBS:power
 LIBS:device
@@
 Sheet 10 10
 Title ""
-Date "13 oct 2012"
+Date "14 oct 2012"
 Rev ""
 Comp ""
@@
 Wire Wire Line
 	3250 5200 2350 5200
-Wire Wire Line
-	8250 5800 8050 5800
-Wire Wire Line
-	8050 5800 8050 5950
 Connection ~ 2550 5200
 Wire Wire Line
@@
 	2650 5200 2650 5050
 Connection ~ 2650 5200
-Wire Wire Line
-	8250 5600 8050 5600
-Wire Wire Line
-	8050 5600 8050 5500
 Wire Wire Line
 	1500 6900 1500 7100
@@
 	1    0    0    -1
 $EndComp
-$Comp
-L GND #PWR0133
-U 1 1 4EBEE96C
-P 8050 5950
-F 0 "#PWR0133" H 8050 5950 30  0001 C CNN
-F 1 "GND" H 8050 5880 30  0001 C CNN
-	1    8050 5950
-	1    0    0    -1
-$EndComp
-$Comp
-L +24V #PWR0134
-U 1 1 4EBEE964
-P 8050 5500
-F 0 "#PWR0134" H 8050 5450 20  0001 C CNN
-F 1 "+24V" H 8050 5600 30  0000 C CNN
-	1    8050 5500
-	1    0    0    -1
-$EndComp
-$Comp
-L CONN_2 P27
-U 1 1 4EBEE955
-P 8600 5700
-F 0 "P27" V 8550 5700 40  0000 C CNN
-F 1 "Power" V 8650 5700 40  0000 C CNN
-	1    8600 5700
-	1    0    0    -1
-$EndComp
