File: laserctrl/watchdog.sch (KiCad schematic (older format))
At the start: 7 parts, among them CON1 AVR-ISP-6, IC3 ATMEGA328-A, X3 10MHz

Commit message: Added connections to the watchdog
Parts:
- removed IC3: ATMEGA328-A, TQFP32, symbol ATMEGA328-A
- added C? (x3): 100nF, symbol C
- added IC?: ATMEGA328P-A, TQFP32, symbol ATMEGA328P-A
- CON1: value AVR-ISP-6 -> WD-ISP
Connections:
- net labels added: +3.3V, MISO_wd, MOSI_wd, SCK_wd, ~Reset_wd
- net labels removed: +5V, MISO, MOSI, SCK, ~Reset, ~reset
- wire segments 27 -> 54
Other:
- moved on the sheet: C41, C42, C43, CON1, R63, X3

Commit message: Started assigning footprints
Parts:
- gave numbers to parts that had none: 4
- renumbered C43 to C41, C41 to C46, R63 to R65
Changed lines of the file:
@@
-EESchema Schematic File Version 2  date 2011-11-07T21:51:12 CET
+EESchema Schematic File Version 2  date 2011-11-07T23:14:52 CET
 LIBS:power
 LIBS:device
@@
 $EndDescr
 Wire Wire Line
-	2000 3400 2000 3450
+	2000 3450 2000 3400
 Wire Wire Line
 	2000 3400 1400 3400
@@
 Connection ~ 1700 3400
 $Comp
-L GND #PWR?
+L GND #PWR090
 U 1 1 4EB84218
 P 1700 4000
-F 0 "#PWR?" H 1700 4000 30  0001 C CNN
+F 0 "#PWR090" H 1700 4000 30  0001 C CNN
 F 1 "GND" H 1700 3930 30  0001 C CNN
 	1    1700 4000
@@
 $EndComp
 $Comp
-L +3.3V #PWR?
+L +3.3V #PWR091
 U 1 1 4EB84214
 P 1700 3300
-F 0 "#PWR?" H 1700 3260 30  0001 C CNN
+F 0 "#PWR091" H 1700 3260 30  0001 C CNN
 F 1 "+3.3V" H 1700 3410 30  0000 C CNN
 	1    1700 3300
@@
 $EndComp
 $Comp
-L C C?
+L C C45
 U 1 1 4EB84209
 P 2000 3650
-F 0 "C?" H 2050 3750 50  0000 L CNN
+F 0 "C45" H 2050 3750 50  0000 L CNN
 F 1 "100nF" H 2050 3550 50  0000 L CNN
 	1    2000 3650
@@
 $EndComp
 $Comp
-L C C?
+L C C44
 U 1 1 4EB84203
 P 1700 3650
-F 0 "C?" H 1750 3750 50  0000 L CNN
+F 0 "C44" H 1750 3750 50  0000 L CNN
 F 1 "100nF" H 1750 3550 50  0000 L CNN
 	1    1700 3650
@@
 $EndComp
 $Comp
-L C C?
+L C C43
 U 1 1 4EB841FC
 P 1400 3650
-F 0 "C?" H 1450 3750 50  0000 L CNN
+F 0 "C43" H 1450 3750 50  0000 L CNN
 F 1 "100nF" H 1450 3550 50  0000 L CNN
 	1    1400 3650
@@
 $EndComp
 $Comp
-L GND #PWR?
+L GND #PWR092
 U 1 1 4EB84050
 P 4450 4900
-F 0 "#PWR?" H 4450 4900 30  0001 C CNN
+F 0 "#PWR092" H 4450 4900 30  0001 C CNN
 F 1 "GND" H 4450 4830 30  0001 C CNN
 	1    4450 4900
@@
 $EndComp
 $Comp
-L +3.3V #PWR?
+L +3.3V #PWR093
 U 1 1 4EB84034
 P 4350 1700
-F 0 "#PWR?" H 4350 1660 30  0001 C CNN
+F 0 "#PWR093" H 4350 1660 30  0001 C CNN
 F 1 "+3.3V" H 4350 1810 30  0000 C CNN
 	1    4350 1700
@@
 MISO_wd
 $Comp
-L +3.3V #PWR?
+L +3.3V #PWR094
 U 1 1 4EB83FCF
 P 2450 1950
-F 0 "#PWR?" H 2450 1910 30  0001 C CNN
+F 0 "#PWR094" H 2450 1910 30  0001 C CNN
 F 1 "+3.3V" H 2450 2060 30  0000 C CNN
 	1    2450 1950
@@
 $EndComp
 $Comp
-L GND #PWR?
+L GND #PWR095
 U 1 1 4EB83F3F
 P 3500 3200
-F 0 "#PWR?" H 3500 3200 30  0001 C CNN
+F 0 "#PWR095" H 3500 3200 30  0001 C CNN
 F 1 "GND" H 3500 3130 30  0001 C CNN
 	1    3500 3200
@@
 $EndComp
 $Comp
-L +3.3V #PWR?
+L +3.3V #PWR096
 U 1 1 4EB83F32
 P 3500 1800
-F 0 "#PWR?" H 3500 1760 30  0001 C CNN
+F 0 "#PWR096" H 3500 1760 30  0001 C CNN
 F 1 "+3.3V" H 3500 1910 30  0000 C CNN
 	1    3500 1800
@@
 $EndComp
 $Comp
-L GND #PWR?
+L GND #PWR097
 U 1 1 4EB83ED6
 P 2600 4100
-F 0 "#PWR?" H 2600 4100 30  0001 C CNN
+F 0 "#PWR097" H 2600 4100 30  0001 C CNN
 F 1 "GND" H 2600 4030 30  0001 C CNN
 	1    2600 4100
@@
 $EndComp
 $Comp
-L ATMEGA328P-A IC?
+L ATMEGA328P-A IC3
 U 1 1 4EB83DB6
 P 4650 3250
-F 0 "IC?" H 4700 4500 50  0000 L BNN
+F 0 "IC3" H 4700 4500 50  0000 L BNN
 F 1 "ATMEGA328P-A" H 4850 1850 50  0000 L BNN
 F 2 "TQFP32" H 4100 1900 50  0001 C CNN
@@
 TXD
 $Comp
-L C C43
+L C C41
 U 1 1 4EA3E4C4
 P 3500 2900
-F 0 "C43" H 3550 3000 50  0000 L CNN
+F 0 "C41" H 3550 3000 50  0000 L CNN
 F 1 "100nF" H 3550 2800 50  0000 L CNN
 	1    3500 2900
@@
 $EndComp
 $Comp
-L R R63
+L R R65
 U 1 1 4EA3E4C2
 P 3500 2150
-F 0 "R63" V 3580 2150 50  0000 C CNN
+F 0 "R65" V 3580 2150 50  0000 C CNN
 F 1 "10k" V 3500 2150 50  0000 C CNN
 	1    3500 2150
@@
 U 1 1 4EA3E4C0
 P 3500 3700
-F 0 "X3" H 3500 3850 60  0000 C CNN
-F 1 "10MHz" H 3500 3550 60  0000 C CNN
+F 0 "X3" V 3500 3850 60  0000 C CNN
+F 1 "10MHz" V 3350 3500 60  0000 C CNN
 	1    3500 3700
 	0    1    1    0
 $EndComp
 $Comp
-L C C41
+L C C46
 U 1 1 4EA3E4BF
 P 2950 4000
-F 0 "C41" H 3000 4100 50  0000 L CNN
-F 1 "15pF" H 3000 3900 50  0000 L CNN
+F 0 "C46" V 2850 4150 50  0000 L CNN
+F 1 "15pF" V 2850 3800 50  0000 L CNN
 	1    2950 4000
 	0    1    1    0
@@
 U 1 1 4EA3E4BE
 P 2950 3400
-F 0 "C42" H 3000 3500 50  0000 L CNN
-F 1 "15pF" H 3000 3300 50  0000 L CNN
+F 0 "C42" V 2850 3550 50  0000 L CNN
+F 1 "15pF" V 2850 3200 50  0000 L CNN
 	1    2950 3400
 	0    1    1    0
@@
 ~Reset_wd
 $Comp
-L GND #PWR93
+L GND #PWR098
 U 1 1 4EA3E4B9
 P 2450 2450
-F 0 "#PWR93" H 2450 2450 30  0001 C CNN
+F 0 "#PWR098" H 2450 2450 30  0001 C CNN
 F 1 "GND" H 2450 2380 30  0001 C CNN
 	1    2450 2450
