File: laserctrl/chiller-if.sch (KiCad schematic (older format))
At the start: 1 part

Commit message: Added a todo list so I don't forget the last bits and tried annotating different ways
Parts:
- gave numbers to parts that had none: 1
Changed lines of the file:
@@
-EESchema Schematic File Version 2  date 2011-11-06T20:55:52 CET
+EESchema Schematic File Version 2  date 2011-11-06T22:48:15 CET
 LIBS:power
 LIBS:device
@@
 	2950 1800 2900 1800
 Wire Wire Line
-	2100 1700 1950 1700
+	2100 1700 1800 1700
 Wire Wire Line
 	2900 1700 3100 1700
@@
 	3100 1700 3100 1650
 Wire Wire Line
-	1950 1800 2100 1800
+	1800 1800 2100 1800
 Wire Wire Line
 	2900 1900 2950 1900
@@
 Connection ~ 2950 2100
 $Comp
-L +24V #PWR?
+L +24V #PWR15
 U 1 1 4EB6DCEF
 P 1900 2200
-F 0 "#PWR?" H 1900 2150 20  0001 C CNN
+F 0 "#PWR15" H 1900 2150 20  0001 C CNN
 F 1 "+24V" H 1900 2300 30  0000 C CNN
 	1    1900 2200
@@
 $EndComp
 $Comp
-L GND #PWR?
+L GND #PWR14
 U 1 1 4EB6DCC0
 P 1900 1950
-F 0 "#PWR?" H 1900 1950 30  0001 C CNN
+F 0 "#PWR14" H 1900 1950 30  0001 C CNN
 F 1 "GND" H 1900 1880 30  0001 C CNN
 	1    1900 1950
 	1    0    0    -1
 $EndComp
-Text HLabel 1950 1800 0    50   Output ~ 0
+Text HLabel 1800 1800 0    50   Output ~ 0
 RXD
-Text HLabel 1950 1700 0    50   Input ~ 0
+Text HLabel 1800 1700 0    50   Input ~ 0
 TXD
 $Comp
-L +3.3V #PWR?
+L +3.3V #PWR12
 U 1 1 4EB6DB66
 P 3100 1650
-F 0 "#PWR?" H 3100 1610 30  0001 C CNN
+F 0 "#PWR12" H 3100 1610 30  0001 C CNN
 F 1 "+3.3V" H 3100 1760 30  0000 C CNN
 	1    3100 1650
@@
 $EndComp
 $Comp
-L GND #PWR?
+L GND #PWR13
 U 1 1 4EB6DB2E
 P 3100 1850
-F 0 "#PWR?" H 3100 1850 30  0001 C CNN
+F 0 "#PWR13" H 3100 1850 30  0001 C CNN
 F 1 "GND" H 3100 1780 30  0001 C CNN
 	1    3100 1850
@@
 $EndComp
 $Comp
-L CONN_5X2 P?
+L CONN_5X2 P2
 U 1 1 4EB6DB27
 P 2500 1900
-F 0 "P?" H 2500 2200 60  0000 C CNN
+F 0 "P2" H 2500 2200 60  0000 C CNN
 F 1 "CONN_5X2" V 2500 1900 50  0000 C CNN
 	1    2500 1900

Commit message: Started assigning footprints
Parts:
- P4: renamed from P2; value CONN_5X2 -> Chiller
Changed lines of the file:
@@
-EESchema Schematic File Version 2  date 2011-11-07T21:51:12 CET
+EESchema Schematic File Version 2  date 2011-11-07T23:14:52 CET
 LIBS:power
 LIBS:device
@@
 $Descr A4 11700 8267
 encoding utf-8
-Sheet 2 12
+Sheet 3 12
 Title ""
 Date "7 nov 2011"
@@
 Connection ~ 2050 2200
 Wire Wire Line
-	1900 2200 2050 2200
+	2950 2200 1900 2200
 Wire Wire Line
-	2050 2200 2950 2200
+	2950 2000 2900 2000
 Wire Wire Line
-	2900 2000 2950 2000
-Wire Wire Line
-	2950 2000 2950 2100
-Wire Wire Line
-	2950 2100 2950 2200
+	2950 2200 2950 2000
 Wire Wire Line
 	2050 2200 2050 2100
@@
 	2050 2100 2100 2100
 Wire Wire Line
-	2100 1900 2050 1900
-Wire Wire Line
-	2050 1900 1900 1900
+	2100 1900 1900 1900
 Wire Wire Line
 	1900 1900 1900 1950
 Wire Wire Line
-	3100 1850 3100 1800
+	3100 1800 3100 1850
 Wire Wire Line
-	3100 1800 2950 1800
-Wire Wire Line
-	2950 1800 2900 1800
+	2900 1800 3100 1800
 Wire Wire Line
 	2100 1700 1800 1700
@@
 Connection ~ 2950 2100
 $Comp
-L +24V #PWR15
+L +24V #PWR016
 U 1 1 4EB6DCEF
 P 1900 2200
-F 0 "#PWR15" H 1900 2150 20  0001 C CNN
+F 0 "#PWR016" H 1900 2150 20  0001 C CNN
 F 1 "+24V" H 1900 2300 30  0000 C CNN
 	1    1900 2200
@@
 $EndComp
 $Comp
-L GND #PWR14
+L GND #PWR017
 U 1 1 4EB6DCC0
 P 1900 1950
-F 0 "#PWR14" H 1900 1950 30  0001 C CNN
+F 0 "#PWR017" H 1900 1950 30  0001 C CNN
 F 1 "GND" H 1900 1880 30  0001 C CNN
 	1    1900 1950
@@
 TXD
 $Comp
-L +3.3V #PWR12
+L +3.3V #PWR018
 U 1 1 4EB6DB66
 P 3100 1650
-F 0 "#PWR12" H 3100 1610 30  0001 C CNN
+F 0 "#PWR018" H 3100 1610 30  0001 C CNN
 F 1 "+3.3V" H 3100 1760 30  0000 C CNN
 	1    3100 1650
@@
 $EndComp
 $Comp
-L GND #PWR13
+L GND #PWR019
 U 1 1 4EB6DB2E
 P 3100 1850
-F 0 "#PWR13" H 3100 1850 30  0001 C CNN
+F 0 "#PWR019" H 3100 1850 30  0001 C CNN
 F 1 "GND" H 3100 1780 30  0001 C CNN
 	1    3100 1850
@@
 $EndComp
 $Comp
-L CONN_5X2 P2
+L CONN_5X2 P4
 U 1 1 4EB6DB27
 P 2500 1900
-F 0 "P2" H 2500 2200 60  0000 C CNN
-F 1 "CONN_5X2" V 2500 1900 50  0000 C CNN
+F 0 "P4" H 2500 2200 60  0000 C CNN
+F 1 "Chiller" V 2500 1900 50  0000 C CNN
 	1    2500 1900
 	1    0    0    -1
