File: laserctrl/relays.sch (KiCad schematic (older format))
At the start: 8 parts

Commit message: Started assigning footprints
Parts:
- R10, R9: renamed from R?; value R -> 3k3
- gave numbers to parts that had none: 6
Changed lines of the file:
@@
-EESchema Schematic File Version 2  date 2011-11-07T21:51:12 CET
+EESchema Schematic File Version 2  date 2011-11-07T23:14:52 CET
 LIBS:power
 LIBS:device
@@
 $EndDescr
 $Comp
-L R R?
+L R R10
 U 1 1 4EB83234
 P 2500 3650
-F 0 "R?" V 2580 3650 50  0000 C CNN
-F 1 "R" V 2500 3650 50  0000 C CNN
+F 0 "R10" V 2580 3650 50  0000 C CNN
+F 1 "3k3" V 2500 3650 50  0000 C CNN
 	1    2500 3650
 	0    1    1    0
 $EndComp
 $Comp
-L NPN Q?
+L NPN Q2
 U 1 1 4EB83233
 P 3050 3650
-F 0 "Q?" H 3050 3500 50  0000 R CNN
+F 0 "Q2" H 3050 3500 50  0000 R CNN
 F 1 "BC817" H 3050 3800 50  0000 R CNN
 	1    3050 3650
@@
 $EndComp
 $Comp
-L GND #PWR?
+L GND #PWR012
 U 1 1 4EB83232
 P 3150 3900
-F 0 "#PWR?" H 3150 3900 30  0001 C CNN
+F 0 "#PWR012" H 3150 3900 30  0001 C CNN
 F 1 "GND" H 3150 3830 30  0001 C CNN
 	1    3150 3900
@@
 $EndComp
 $Comp
-L CONN_2 P?
+L CONN_2 P3
 U 1 1 4EB83231
 P 3750 3300
-F 0 "P?" V 3700 3300 40  0000 C CNN
+F 0 "P3" V 3700 3300 40  0000 C CNN
 F 1 "Assist Air" V 3800 3300 40  0000 C CNN
 	1    3750 3300
@@
 $EndComp
 $Comp
-L DIODE D?
+L DIODE D2
 U 1 1 4EB83230
 P 3150 3150
-F 0 "D?" H 3150 3250 40  0000 C CNN
+F 0 "D2" H 3150 3250 40  0000 C CNN
 F 1 "DIODE" H 3150 3050 40  0000 C CNN
 	1    3150 3150
@@
 $EndComp
 $Comp
-L +24V #PWR?
+L +24V #PWR013
 U 1 1 4EB8322F
 P 3150 2850
-F 0 "#PWR?" H 3150 2800 20  0001 C CNN
+F 0 "#PWR013" H 3150 2800 20  0001 C CNN
 F 1 "+24V" H 3150 2950 30  0000 C CNN
 	1    3150 2850
@@
 Connection ~ 3150 2900
 Wire Wire Line
-	3400 2900 3150 2900
+	3150 2900 3400 2900
 Wire Wire Line
-	3400 3200 3400 2900
+	3400 2900 3400 3200
 Wire Wire Line
 	2850 3650 2750 3650
@@
 Exhaust
 $Comp
-L +24V #PWR?
+L +24V #PWR014
 U 1 1 4EB83187
 P 3150 1400
-F 0 "#PWR?" H 3150 1350 20  0001 C CNN
+F 0 "#PWR014" H 3150 1350 20  0001 C CNN
 F 1 "+24V" H 3150 1500 30  0000 C CNN
 	1    3150 1400
@@
 $EndComp
 $Comp
-L DIODE D?
+L DIODE D1
 U 1 1 4EB83128
 P 3150 1700
-F 0 "D?" H 3150 1800 40  0000 C CNN
+F 0 "D1" H 3150 1800 40  0000 C CNN
 F 1 "DIODE" H 3150 1600 40  0000 C CNN
 	1    3150 1700
@@
 $EndComp
 $Comp
-L CONN_2 P?
+L CONN_2 P2
 U 1 1 4EB83119
 P 3750 1850
-F 0 "P?" V 3700 1850 40  0000 C CNN
+F 0 "P2" V 3700 1850 40  0000 C CNN
 F 1 "Exhaust" V 3800 1850 40  0000 C CNN
 	1    3750 1850
@@
 $EndComp
 $Comp
-L GND #PWR?
+L GND #PWR015
 U 1 1 4EB830F3
 P 3150 2450
-F 0 "#PWR?" H 3150 2450 30  0001 C CNN
+F 0 "#PWR015" H 3150 2450 30  0001 C CNN
 F 1 "GND" H 3150 2380 30  0001 C CNN
 	1    3150 2450
@@
 $EndComp
 $Comp
-L NPN Q?
+L NPN Q1
 U 1 1 4EB830E3
 P 3050 2200
-F 0 "Q?" H 3050 2050 50  0000 R CNN
+F 0 "Q1" H 3050 2050 50  0000 R CNN
 F 1 "BC817" H 3050 2350 50  0000 R CNN
 	1    3050 2200
@@
 $EndComp
 $Comp
-L R R?
+L R R9
 U 1 1 4EB830BA
 P 2500 2200
-F 0 "R?" V 2580 2200 50  0000 C CNN
-F 1 "R" V 2500 2200 50  0000 C CNN
+F 0 "R9" V 2580 2200 50  0000 C CNN
+F 1 "3k3" V 2500 2200 50  0000 C CNN
 	1    2500 2200
 	0    1    1    0
