File: laserctrl/driver.sch (KiCad schematic (older format))
At the start: 37 parts, among them IC7 DRV8811, P10 CONN_4

Commit message: Added a todo list so I don't forget the last bits and tried annotating different ways
Parts:
- gave numbers to parts that had none: 22
- renumbered C34 to C13, C39 to C15, C37 to C16, C33 to C21, C38 to C22, C35 to C23, C36 to C24, IC7 to IC1, JP7 to JP1, JP8 to JP2, R28 to R44, R29 to R45, R30 to R46, R31 to R47
Connections:
- net +3.3V: no longer IC1.17 (~RESET)
- new net ~RESET: IC1.17 (~RESET)

Commit message: Started assigning footprints
Parts:
- P12: renamed from P10; value CONN_4 -> stepper
- P13: renamed from P11; value CONN_2 -> min
- P14: renamed from P12; value CONN_2 -> max
- renumbered D17 to D19, D18 to D20, D19 to D21, D20 to D22, D21 to D23, D22 to D24, R41 to R43, R42 to R44, R43 to R45, R44 to R46, R45 to R47, R46 to R48, R47 to R49, R48 to R50, R49 to R51, R50 to R52, R51 to R53

Commit message: Started some cleaning up
Parts:
- removed C14: 10uF, symbol C
- C18: value 10uF -> 10uF/35V
- C19: value 220uF -> 330uF/35V
Connections:
- wire segments 102 -> 100
Other:
- moved on the sheet: JP1, JP2

Commit message: Use double-shottky diodes in stead of tons of discrete miniMELFs
Parts:
- removed C26: 10nF, symbol C
- removed D19, D20, D23, D24: DIODE, symbol DIODE
- removed D22: LED, symbol LED
- removed R52: 330, symbol R
- removed R53: 1k, symbol R
- added C28: 10nF, symbol C
- added D26: LED, symbol LED
- added D28, D29: BAT 54S, symbol DIODE2
- added R76: 330, symbol R
- added R86: 1k, symbol R
- JP1: value JUMPER3 -> USM0
- JP2: value JUMPER3 -> USM1
Connections:
- wire segments 100 -> 98
