File: laserctrl/driver.sch (KiCad schematic (older format))
At the start: 27 parts, among them IC1 DRV8811, P12 stepper, P13 min, P14 max

Commit message: Generated the BOM and figured out what parts to buy at ELFA and Mouser
Changed lines of the file:
@@
-EESchema Schematic File Version 2  date 2011-11-28T22:17:03 CET
+EESchema Schematic File Version 2  date 2011-12-03T21:12:32 CET
 LIBS:power
 LIBS:device
@@
 $Descr A4 11700 8267
 encoding utf-8
-Sheet 9 10
+Sheet 8 10
 Title ""
-Date "27 nov 2011"
+Date "3 dec 2011"
 Rev ""
 Comp ""
@@
 Comment4 ""
 $EndDescr
+Connection ~ 2250 6500
 Wire Wire Line
 	6800 3350 6650 3350
@@
 AR Path="/4EA1D353/4EBAE0A4" Ref="C14"  Part="1"
 AR Path="/4EA1F56E/4EBAE0A4" Ref="C26"  Part="1"
-F 0 "C28" H 4100 7450 50  0000 L CNN
+F 0 "C26" H 4100 7450 50  0000 L CNN
 F 1 "10nF" H 4050 7250 50  0000 L CNN
 	1    4250 7350
@@
 AR Path="/4EA1D353/4EBAE0A3" Ref="#PWR085"  Part="1"
 AR Path="/4EA1F56E/4EBAE0A3" Ref="#PWR0106"  Part="1"
-F 0 "#PWR0118" H 4450 7650 30  0001 C CNN
+F 0 "#PWR0106" H 4450 7650 30  0001 C CNN
 F 1 "GND" H 4450 7580 30  0001 C CNN
 	1    4450 7650
@@
 AR Path="/4EA1D353/4EBAE0A2" Ref="R63"  Part="1"
 AR Path="/4EA1F56E/4EBAE0A2" Ref="R75"  Part="1"
-F 0 "R86" V 4330 6800 50  0000 C CNN
+F 0 "R75" V 4330 6800 50  0000 C CNN
 F 1 "1k" V 4250 6800 50  0000 C CNN
 	1    4250 6800
@@
 AR Path="/4EA1D353/4EBAE09F" Ref="#PWR086"  Part="1"
 AR Path="/4EA1F56E/4EBAE09F" Ref="#PWR0107"  Part="1"
-F 0 "#PWR0119" H 4450 6410 30  0001 C CNN
+F 0 "#PWR0107" H 4450 6410 30  0001 C CNN
 F 1 "+3.3V" H 4450 6560 30  0000 C CNN
 	1    4450 6450
@@
 AR Path="/4EA1D353/4EBAE09E" Ref="D22"  Part="1"
 AR Path="/4EA1F56E/4EBAE09E" Ref="D25"  Part="1"
-F 0 "D29" H 4300 6900 60  0000 C CNN
+F 0 "D25" H 4300 6900 60  0000 C CNN
 F 1 "BAT 54S" H 4150 7000 60  0000 C CNN
 	1    4450 7150
@@
 AR Path="/4EA1D353/4EBAE046" Ref="D20"  Part="1"
 AR Path="/4EA1F56E/4EBAE046" Ref="D24"  Part="1"
-F 0 "D28" H 2150 6900 60  0000 C CNN
+F 0 "D24" H 2150 6900 60  0000 C CNN
 F 1 "BAT 54S" H 2000 7000 60  0000 C CNN
 	1    2250 7150
@@
 AR Path="/4EA1F56E/4EB45B46" Ref="#PWR0108"  Part="1"
 AR Path="/4EA1D331/4EB45B46" Ref="#PWR0120"  Part="1"
-F 0 "#PWR0120" H 6850 1800 30  0001 C CNN
+F 0 "#PWR0108" H 6850 1800 30  0001 C CNN
 F 1 "GND" H 6850 1730 30  0001 C CNN
 	1    6850 1800
@@
 AR Path="/4EA1F56E/4EB45B01" Ref="C52"  Part="1"
 AR Path="/4EA1D331/4EB45B01" Ref="C66"  Part="1"
-F 0 "C66" H 6900 1600 50  0000 L CNN
+F 0 "C52" H 6900 1600 50  0000 L CNN
 F 1 "10uF/35V" H 6900 1400 50  0000 L CNN
 	1    6850 1500
@@
 AR Path="/4EA1F56E/4EB45AF6" Ref="C51"  Part="1"
 AR Path="/4EA1D331/4EB45AF6" Ref="C65"  Part="1"
-F 0 "C65" H 6550 1600 50  0000 L CNN
+F 0 "C51" H 6550 1600 50  0000 L CNN
 F 1 "100nF" H 6550 1400 50  0000 L CNN
 	1    6500 1500
@@
 AR Path="/4EA1F56E/4EB45A38" Ref="#PWR0109"  Part="1"
 AR Path="/4EA1D331/4EB45A38" Ref="#PWR0121"  Part="1"
-F 0 "#PWR0121" H 2250 6460 30  0001 C CNN
+F 0 "#PWR0109" H 2250 6460 30  0001 C CNN
 F 1 "+3.3V" H 2250 6610 30  0000 C CNN
 	1    2250 6500
@@
 AR Path="/4EA1F56E/4EB45A35" Ref="R74"  Part="1"
 AR Path="/4EA1D331/4EB45A35" Ref="R85"  Part="1"
-F 0 "R85" V 2130 6800 50  0000 C CNN
+F 0 "R74" V 2130 6800 50  0000 C CNN
 F 1 "1k" V 2050 6800 50  0000 C CNN
 	1    2050 6800
@@
 AR Path="/4EA1F56E/4EB45A34" Ref="P19"  Part="1"
 AR Path="/4EA1D331/4EB45A34" Ref="P22"  Part="1"
-F 0 "P22" V 2800 7250 40  0000 C CNN
+F 0 "P19" V 2800 7250 40  0000 C CNN
 F 1 "min" V 2900 7250 40  0000 C CNN
 	1    2850 7250
@@
 AR Path="/4EA1F56E/4EB45A33" Ref="#PWR0110"  Part="1"
 AR Path="/4EA1D331/4EB45A33" Ref="#PWR0122"  Part="1"
-F 0 "#PWR0122" H 2250 7650 30  0001 C CNN
+F 0 "#PWR0110" H 2250 7650 30  0001 C CNN
 F 1 "GND" H 2250 7580 30  0001 C CNN
 	1    2250 7650
@@
 AR Path="/4EA1F56E/4EB45A32" Ref="C59"  Part="1"
 AR Path="/4EA1D331/4EB45A32" Ref="C73"  Part="1"
-F 0 "C73" H 1900 7450 50  0000 L CNN
+F 0 "C59" H 1900 7450 50  0000 L CNN
 F 1 "10nF" H 1850 7250 50  0000 L CNN
 	1    2050 7350
@@
 AR Path="/4EA1F56E/4EB4496F" Ref="P20"  Part="1"
 AR Path="/4EA1D331/4EB4496F" Ref="P23"  Part="1"
-F 0 "P23" V 5000 7250 40  0000 C CNN
+F 0 "P20" V 5000 7250 40  0000 C CNN
 F 1 "max" V 5100 7250 40  0000 C CNN
 	1    5050 7250
@@
 AR Path="/4EA1F56E/4EAD2C72" Ref="#PWR0111"  Part="1"
 AR Path="/4EA1D331/4EAD2C72" Ref="#PWR0123"  Part="1"
-F 0 "#PWR0123" H 2100 3760 30  0001 C CNN
+F 0 "#PWR0111" H 2100 3760 30  0001 C CNN
 F 1 "+3.3V" H 2100 3910 30  0000 C CNN
 	1    2100 3800
@@
 AR Path="/4EA1F56E/4EAD2C5D" Ref="#PWR0112"  Part="1"
 AR Path="/4EA1D331/4EAD2C5D" Ref="#PWR0124"  Part="1"
-F 0 "#PWR0124" H 4250 1010 30  0001 C CNN
+F 0 "#PWR0112" H 4250 1010 30  0001 C CNN
 F 1 "+3.3V" H 4250 1160 30  0000 C CNN
 	1    4250 1050
@@
 AR Path="/4EA1F56E/4EAD2C05" Ref="#PWR0113"  Part="1"
 AR Path="/4EA1D331/4EAD2C05" Ref="#PWR0125"  Part="1"
-F 0 "#PWR0125" H 3350 4600 30  0001 C CNN
+F 0 "#PWR0113" H 3350 4600 30  0001 C CNN
 F 1 "GND" H 3350 4530 30  0001 C CNN
 	1    3350 4600
@@
 AR Path="/4EA1F56E/4EAD2BEA" Ref="C54"  Part="1"
 AR Path="/4EA1D331/4EAD2BEA" Ref="C68"  Part="1"
-F 0 "C68" H 3400 4400 50  0000 L CNN
+F 0 "C54" H 3400 4400 50  0000 L CNN
 F 1 "100nF" H 3100 4200 50  0000 L CNN
 	1    3350 4300
@@
 AR Path="/4EA1F56E/4EAD2BE0" Ref="R66"  Part="1"
 AR Path="/4EA1D331/4EAD2BE0" Ref="R77"  Part="1"
-F 0 "R77" V 3080 4000 50  0000 C CNN
+F 0 "R66" V 3080 4000 50  0000 C CNN
 F 1 "10k" V 3000 4000 50  0000 C CNN
 	1    3000 4000
@@
 AR Path="/4EA1F56E/4EAD2AB6" Ref="R67"  Part="1"
 AR Path="/4EA1D331/4EAD2AB6" Ref="R78"  Part="1"
-F 0 "R78" V 2180 4150 50  0000 C CNN
+F 0 "R67" V 2180 4150 50  0000 C CNN
 F 1 "10k" V 2100 4150 50  0000 C CNN
 	1    2100 4150
@@
 AR Path="/4EA1F56E/4EAD2AA2" Ref="R68"  Part="1"
 AR Path="/4EA1D331/4EAD2AA2" Ref="R79"  Part="1"
-F 0 "R79" V 2180 4750 50  0000 C CNN
+F 0 "R68" V 2180 4750 50  0000 C CNN
 F 1 "10k" V 2100 4750 50  0000 C CNN
 	1    2100 4750
@@
 AR Path="/4EA1F56E/4EA1E74B" Ref="IC4"  Part="1"
 AR Path="/4EA1D331/4EA1E74B" Ref="IC5"  Part="1"
-F 0 "IC5" H 5050 3500 60  0000 C CNN
+F 0 "IC4" H 5050 3500 60  0000 C CNN
 F 1 "DRV8811" H 5050 3300 60  0000 C CNN
 	1    5050 3300
@@
 AR Path="/4EA1F56E/4EA1F353" Ref="#PWR0114"  Part="1"
 AR Path="/4EA1D331/4EA1F353" Ref="#PWR0126"  Part="1"
-F 0 "#PWR0126" H 2100 5100 30  0001 C CNN
+F 0 "#PWR0114" H 2100 5100 30  0001 C CNN
 F 1 "GND" H 2100 5030 30  0001 C CNN
 	1    2100 5100
@@
 AR Path="/4EA1F56E/4EA1F336" Ref="C55"  Part="1"
 AR Path="/4EA1D331/4EA1F336" Ref="C69"  Part="1"
-F 0 "C69" H 1700 4850 50  0000 L CNN
+F 0 "C55" H 1700 4850 50  0000 L CNN
 F 1 "100nF" H 1600 4650 50  0000 L CNN
 	1    1850 4750
@@
 AR Path="/4EA1F56E/4EA1F182" Ref="P18"  Part="1"
 AR Path="/4EA1D331/4EA1F182" Ref="P21"  Part="1"
-F 0 "P21" V 7100 3300 50  0000 C CNN
+F 0 "P18" V 7100 3300 50  0000 C CNN
 F 1 "stepper" V 7200 3300 50  0000 C CNN
 	1    7150 3300
@@
 AR Path="/4EA1F56E/4EA1EDD7" Ref="#PWR0115"  Part="1"
 AR Path="/4EA1D331/4EA1EDD7" Ref="#PWR0127"  Part="1"
-F 0 "#PWR0127" H 4750 5600 30  0001 C CNN
+F 0 "#PWR0115" H 4750 5600 30  0001 C CNN
 F 1 "GND" H 4750 5530 30  0001 C CNN
 	1    4750 5600
@@
 AR Path="/4EA1F56E/4EA1EDA2" Ref="R69"  Part="1"
 AR Path="/4EA1D331/4EA1EDA2" Ref="R80"  Part="1"
-F 0 "R80" V 4550 5250 50  0000 C CNN
+F 0 "R69" V 4550 5250 50  0000 C CNN
 F 1 "33k" V 4650 5150 50  0000 C CNN
 	1    4650 5150
@@
 AR Path="/4EA1F56E/4EA1ED9B" Ref="C57"  Part="1"
 AR Path="/4EA1D331/4EA1ED9B" Ref="C71"  Part="1"
-F 0 "C71" V 4750 5300 50  0000 L CNN
+F 0 "C57" V 4750 5300 50  0000 L CNN
 F 1 "1nF" V 4750 5000 50  0000 L CNN
 	1    4850 5150
@@
 AR Path="/4EA1F56E/4EA1E91D" Ref="C58"  Part="1"
 AR Path="/4EA1D331/4EA1E91D" Ref="C72"  Part="1"
-F 0 "C72" V 5150 5300 50  0000 L CNN
+F 0 "C58" V 5150 5300 50  0000 L CNN
 F 1 "1nF" V 5150 5000 50  0000 L CNN
 	1    5250 5150
@@
 AR Path="/4EA1F56E/4EA1E910" Ref="R70"  Part="1"
 AR Path="/4EA1D331/4EA1E910" Ref="R81"  Part="1"
-F 0 "R81" V 4950 5300 50  0000 C CNN
+F 0 "R70" V 4950 5300 50  0000 C CNN
 F 1 "33k" V 5050 5150 50  0000 C CNN
 	1    5050 5150
@@
 AR Path="/4EA1F56E/4EA1E8C1" Ref="R71"  Part="1"
 AR Path="/4EA1D331/4EA1E8C1" Ref="R82"  Part="1"
-F 0 "R82" V 5630 5150 50  0000 C CNN
+F 0 "R71" V 5630 5150 50  0000 C CNN
 F 1 "0R22" V 5550 5150 50  0000 C CNN
 	1    5550 5150
@@
 AR Path="/4EA1F56E/4EA1E8BB" Ref="R72"  Part="1"
 AR Path="/4EA1D331/4EA1E8BB" Ref="R83"  Part="1"
-F 0 "R83" V 5880 5150 50  0000 C CNN
+F 0 "R72" V 5880 5150 50  0000 C CNN
 F 1 "0R22" V 5800 5150 50  0000 C CNN
 	1    5800 5150
@@
 AR Path="/4EA1F56E/4EA1E852" Ref="C56"  Part="1"
 AR Path="/4EA1D331/4EA1E852" Ref="C70"  Part="1"
-F 0 "C70" H 6100 5200 50  0000 L CNN
+F 0 "C56" H 6100 5200 50  0000 L CNN
 F 1 "220nF" H 6100 5000 50  0000 L CNN
 	1    6050 5100
@@
 AR Path="/4EA1F56E/4EA1E80A" Ref="#PWR0116"  Part="1"
 AR Path="/4EA1D331/4EA1E80A" Ref="#PWR0128"  Part="1"
-F 0 "#PWR0128" H 4450 1850 30  0001 C CNN
+F 0 "#PWR0116" H 4450 1850 30  0001 C CNN
 F 1 "GND" H 4450 1780 30  0001 C CNN
 	1    4450 1850
@@
 AR Path="/4EA1F56E/4EA1E7F2" Ref="C47"  Part="1"
 AR Path="/4EA1D331/4EA1E7F2" Ref="C61"  Part="1"
-F 0 "C61" H 4500 1550 50  0000 L CNN
+F 0 "C47" H 4500 1550 50  0000 L CNN
 F 1 "100nF" H 4500 1350 50  0000 L CNN
 	1    4450 1450
@@
 AR Path="/4EA1F56E/4EA1E798" Ref="C49"  Part="1"
 AR Path="/4EA1D331/4EA1E798" Ref="C63"  Part="1"
-F 0 "C63" V 5250 1650 50  0000 L CNN
+F 0 "C49" V 5250 1650 50  0000 L CNN
 F 1 "220nF" V 5250 1300 50  0000 L CNN
 	1    5350 1500
@@
 AR Path="/4EA1F56E/4EA1E774" Ref="C50"  Part="1"
 AR Path="/4EA1D331/4EA1E774" Ref="C64"  Part="1"
-F 0 "C64" H 6100 1600 50  0000 L CNN
+F 0 "C50" H 6100 1600 50  0000 L CNN
 F 1 "220nF" H 6100 1400 50  0000 L CNN
 	1    6050 1500
@@
 AR Path="/4EA1F56E/4EA1E764" Ref="#PWR0117"  Part="1"
 AR Path="/4EA1D331/4EA1E764" Ref="#PWR0129"  Part="1"
-F 0 "#PWR0129" H 5850 950 20  0001 C CNN
+F 0 "#PWR0117" H 5850 950 20  0001 C CNN
 F 1 "+24V" H 5850 1100 30  0000 C CNN
 	1    5850 1000

Commit message: Checked footprints and fixed 1 thinko on the ARM and unfucked the transistor foot prints
Changed lines of the file:
@@
-EESchema Schematic File Version 2  date 2011-12-03T21:12:32 CET
+EESchema Schematic File Version 2  date 2011-12-07T22:22:26 CET
 LIBS:power
 LIBS:device
@@
 LIBS:78l00a
 LIBS:conn_11x2
+LIBS:bc807
+LIBS:bc817
 LIBS:laserctrl-cache
 EELAYER 25  0
@@
 $Descr A4 11700 8267
 encoding utf-8
-Sheet 8 10
+Sheet 6 10
 Title ""
-Date "3 dec 2011"
+Date "7 dec 2011"
 Rev ""
 Comp ""
@@
 AR Path="/4EA1D353/4EBAE0A4" Ref="C14"  Part="1"
 AR Path="/4EA1F56E/4EBAE0A4" Ref="C26"  Part="1"
-F 0 "C26" H 4100 7450 50  0000 L CNN
+F 0 "C28" H 4100 7450 50  0000 L CNN
 F 1 "10nF" H 4050 7250 50  0000 L CNN
 	1    4250 7350
@@
 AR Path="/4EA1D353/4EBAE0A3" Ref="#PWR085"  Part="1"
 AR Path="/4EA1F56E/4EBAE0A3" Ref="#PWR0106"  Part="1"
-F 0 "#PWR0106" H 4450 7650 30  0001 C CNN
+F 0 "#PWR0118" H 4450 7650 30  0001 C CNN
 F 1 "GND" H 4450 7580 30  0001 C CNN
 	1    4450 7650
@@
 AR Path="/4EA1D353/4EBAE0A2" Ref="R63"  Part="1"
 AR Path="/4EA1F56E/4EBAE0A2" Ref="R75"  Part="1"
-F 0 "R75" V 4330 6800 50  0000 C CNN
+F 0 "R86" V 4330 6800 50  0000 C CNN
 F 1 "1k" V 4250 6800 50  0000 C CNN
 	1    4250 6800
@@
 AR Path="/4EA1D353/4EBAE09F" Ref="#PWR086"  Part="1"
 AR Path="/4EA1F56E/4EBAE09F" Ref="#PWR0107"  Part="1"
-F 0 "#PWR0107" H 4450 6410 30  0001 C CNN
+F 0 "#PWR0119" H 4450 6410 30  0001 C CNN
 F 1 "+3.3V" H 4450 6560 30  0000 C CNN
 	1    4450 6450
@@
 AR Path="/4EA1D353/4EBAE09E" Ref="D22"  Part="1"
 AR Path="/4EA1F56E/4EBAE09E" Ref="D25"  Part="1"
-F 0 "D25" H 4300 6900 60  0000 C CNN
+F 0 "D29" H 4300 6900 60  0000 C CNN
 F 1 "BAT 54S" H 4150 7000 60  0000 C CNN
 	1    4450 7150
@@
 AR Path="/4EA1D353/4EBAE046" Ref="D20"  Part="1"
 AR Path="/4EA1F56E/4EBAE046" Ref="D24"  Part="1"
-F 0 "D24" H 2150 6900 60  0000 C CNN
+F 0 "D28" H 2150 6900 60  0000 C CNN
 F 1 "BAT 54S" H 2000 7000 60  0000 C CNN
 	1    2250 7150
@@
 AR Path="/4EA1F56E/4EB45B46" Ref="#PWR0108"  Part="1"
 AR Path="/4EA1D331/4EB45B46" Ref="#PWR0120"  Part="1"
-F 0 "#PWR0108" H 6850 1800 30  0001 C CNN
+F 0 "#PWR0120" H 6850 1800 30  0001 C CNN
 F 1 "GND" H 6850 1730 30  0001 C CNN
 	1    6850 1800
@@
 AR Path="/4EA1F56E/4EB45B01" Ref="C52"  Part="1"
 AR Path="/4EA1D331/4EB45B01" Ref="C66"  Part="1"
-F 0 "C52" H 6900 1600 50  0000 L CNN
+F 0 "C66" H 6900 1600 50  0000 L CNN
 F 1 "10uF/35V" H 6900 1400 50  0000 L CNN
 	1    6850 1500
@@
 AR Path="/4EA1F56E/4EB45AF6" Ref="C51"  Part="1"
 AR Path="/4EA1D331/4EB45AF6" Ref="C65"  Part="1"
-F 0 "C51" H 6550 1600 50  0000 L CNN
+F 0 "C65" H 6550 1600 50  0000 L CNN
 F 1 "100nF" H 6550 1400 50  0000 L CNN
 	1    6500 1500
@@
 AR Path="/4EA1F56E/4EB45A38" Ref="#PWR0109"  Part="1"
 AR Path="/4EA1D331/4EB45A38" Ref="#PWR0121"  Part="1"
-F 0 "#PWR0109" H 2250 6460 30  0001 C CNN
+F 0 "#PWR0121" H 2250 6460 30  0001 C CNN
 F 1 "+3.3V" H 2250 6610 30  0000 C CNN
 	1    2250 6500
@@
 AR Path="/4EA1F56E/4EB45A35" Ref="R74"  Part="1"
 AR Path="/4EA1D331/4EB45A35" Ref="R85"  Part="1"
-F 0 "R74" V 2130 6800 50  0000 C CNN
+F 0 "R85" V 2130 6800 50  0000 C CNN
 F 1 "1k" V 2050 6800 50  0000 C CNN
 	1    2050 6800
@@
 AR Path="/4EA1F56E/4EB45A34" Ref="P19"  Part="1"
 AR Path="/4EA1D331/4EB45A34" Ref="P22"  Part="1"
-F 0 "P19" V 2800 7250 40  0000 C CNN
+F 0 "P22" V 2800 7250 40  0000 C CNN
 F 1 "min" V 2900 7250 40  0000 C CNN
 	1    2850 7250
@@
 AR Path="/4EA1F56E/4EB45A33" Ref="#PWR0110"  Part="1"
 AR Path="/4EA1D331/4EB45A33" Ref="#PWR0122"  Part="1"
-F 0 "#PWR0110" H 2250 7650 30  0001 C CNN
+F 0 "#PWR0122" H 2250 7650 30  0001 C CNN
 F 1 "GND" H 2250 7580 30  0001 C CNN
 	1    2250 7650
@@
 AR Path="/4EA1F56E/4EB45A32" Ref="C59"  Part="1"
 AR Path="/4EA1D331/4EB45A32" Ref="C73"  Part="1"
-F 0 "C59" H 1900 7450 50  0000 L CNN
+F 0 "C73" H 1900 7450 50  0000 L CNN
 F 1 "10nF" H 1850 7250 50  0000 L CNN
 	1    2050 7350
@@
 AR Path="/4EA1F56E/4EB4496F" Ref="P20"  Part="1"
 AR Path="/4EA1D331/4EB4496F" Ref="P23"  Part="1"
-F 0 "P20" V 5000 7250 40  0000 C CNN
+F 0 "P23" V 5000 7250 40  0000 C CNN
 F 1 "max" V 5100 7250 40  0000 C CNN
 	1    5050 7250
@@
 AR Path="/4EA1F56E/4EAD2C72" Ref="#PWR0111"  Part="1"
 AR Path="/4EA1D331/4EAD2C72" Ref="#PWR0123"  Part="1"
-F 0 "#PWR0111" H 2100 3760 30  0001 C CNN
+F 0 "#PWR0123" H 2100 3760 30  0001 C CNN
 F 1 "+3.3V" H 2100 3910 30  0000 C CNN
 	1    2100 3800
@@
 AR Path="/4EA1F56E/4EAD2C5D" Ref="#PWR0112"  Part="1"
 AR Path="/4EA1D331/4EAD2C5D" Ref="#PWR0124"  Part="1"
-F 0 "#PWR0112" H 4250 1010 30  0001 C CNN
+F 0 "#PWR0124" H 4250 1010 30  0001 C CNN
 F 1 "+3.3V" H 4250 1160 30  0000 C CNN
 	1    4250 1050
@@
 AR Path="/4EA1F56E/4EAD2C05" Ref="#PWR0113"  Part="1"
 AR Path="/4EA1D331/4EAD2C05" Ref="#PWR0125"  Part="1"
-F 0 "#PWR0113" H 3350 4600 30  0001 C CNN
+F 0 "#PWR0125" H 3350 4600 30  0001 C CNN
 F 1 "GND" H 3350 4530 30  0001 C CNN
 	1    3350 4600
@@
 AR Path="/4EA1F56E/4EAD2BEA" Ref="C54"  Part="1"
 AR Path="/4EA1D331/4EAD2BEA" Ref="C68"  Part="1"
-F 0 "C54" H 3400 4400 50  0000 L CNN
+F 0 "C68" H 3400 4400 50  0000 L CNN
 F 1 "100nF" H 3100 4200 50  0000 L CNN
 	1    3350 4300
@@
 AR Path="/4EA1F56E/4EAD2BE0" Ref="R66"  Part="1"
 AR Path="/4EA1D331/4EAD2BE0" Ref="R77"  Part="1"
-F 0 "R66" V 3080 4000 50  0000 C CNN
+F 0 "R77" V 3080 4000 50  0000 C CNN
 F 1 "10k" V 3000 4000 50  0000 C CNN
 	1    3000 4000
@@
 AR Path="/4EA1F56E/4EAD2AB6" Ref="R67"  Part="1"
 AR Path="/4EA1D331/4EAD2AB6" Ref="R78"  Part="1"
-F 0 "R67" V 2180 4150 50  0000 C CNN
+F 0 "R78" V 2180 4150 50  0000 C CNN
 F 1 "10k" V 2100 4150 50  0000 C CNN
 	1    2100 4150
@@
 AR Path="/4EA1F56E/4EAD2AA2" Ref="R68"  Part="1"
 AR Path="/4EA1D331/4EAD2AA2" Ref="R79"  Part="1"
-F 0 "R68" V 2180 4750 50  0000 C CNN
+F 0 "R79" V 2180 4750 50  0000 C CNN
 F 1 "10k" V 2100 4750 50  0000 C CNN
 	1    2100 4750
@@
 AR Path="/4EA1F56E/4EA1E74B" Ref="IC4"  Part="1"
 AR Path="/4EA1D331/4EA1E74B" Ref="IC5"  Part="1"
-F 0 "IC4" H 5050 3500 60  0000 C CNN
+F 0 "IC5" H 5050 3500 60  0000 C CNN
 F 1 "DRV8811" H 5050 3300 60  0000 C CNN
 	1    5050 3300
@@
 AR Path="/4EA1F56E/4EA1F353" Ref="#PWR0114"  Part="1"
 AR Path="/4EA1D331/4EA1F353" Ref="#PWR0126"  Part="1"
-F 0 "#PWR0114" H 2100 5100 30  0001 C CNN
+F 0 "#PWR0126" H 2100 5100 30  0001 C CNN
 F 1 "GND" H 2100 5030 30  0001 C CNN
 	1    2100 5100
@@
 AR Path="/4EA1F56E/4EA1F336" Ref="C55"  Part="1"
 AR Path="/4EA1D331/4EA1F336" Ref="C69"  Part="1"
-F 0 "C55" H 1700 4850 50  0000 L CNN
+F 0 "C69" H 1700 4850 50  0000 L CNN
 F 1 "100nF" H 1600 4650 50  0000 L CNN
 	1    1850 4750
@@
 AR Path="/4EA1F56E/4EA1F182" Ref="P18"  Part="1"
 AR Path="/4EA1D331/4EA1F182" Ref="P21"  Part="1"
-F 0 "P18" V 7100 3300 50  0000 C CNN
+F 0 "P21" V 7100 3300 50  0000 C CNN
 F 1 "stepper" V 7200 3300 50  0000 C CNN
 	1    7150 3300
@@
 AR Path="/4EA1F56E/4EA1EDD7" Ref="#PWR0115"  Part="1"
 AR Path="/4EA1D331/4EA1EDD7" Ref="#PWR0127"  Part="1"
-F 0 "#PWR0115" H 4750 5600 30  0001 C CNN
+F 0 "#PWR0127" H 4750 5600 30  0001 C CNN
 F 1 "GND" H 4750 5530 30  0001 C CNN
 	1    4750 5600
@@
 AR Path="/4EA1F56E/4EA1EDA2" Ref="R69"  Part="1"
 AR Path="/4EA1D331/4EA1EDA2" Ref="R80"  Part="1"
-F 0 "R69" V 4550 5250 50  0000 C CNN
+F 0 "R80" V 4550 5250 50  0000 C CNN
 F 1 "33k" V 4650 5150 50  0000 C CNN
 	1    4650 5150
@@
 AR Path="/4EA1F56E/4EA1ED9B" Ref="C57"  Part="1"
 AR Path="/4EA1D331/4EA1ED9B" Ref="C71"  Part="1"
-F 0 "C57" V 4750 5300 50  0000 L CNN
+F 0 "C71" V 4750 5300 50  0000 L CNN
 F 1 "1nF" V 4750 5000 50  0000 L CNN
 	1    4850 5150
@@
 AR Path="/4EA1F56E/4EA1E91D" Ref="C58"  Part="1"
 AR Path="/4EA1D331/4EA1E91D" Ref="C72"  Part="1"
-F 0 "C58" V 5150 5300 50  0000 L CNN
+F 0 "C72" V 5150 5300 50  0000 L CNN
 F 1 "1nF" V 5150 5000 50  0000 L CNN
 	1    5250 5150
@@
 AR Path="/4EA1F56E/4EA1E910" Ref="R70"  Part="1"
 AR Path="/4EA1D331/4EA1E910" Ref="R81"  Part="1"
-F 0 "R70" V 4950 5300 50  0000 C CNN
+F 0 "R81" V 4950 5300 50  0000 C CNN
 F 1 "33k" V 5050 5150 50  0000 C CNN
 	1    5050 5150
@@
 AR Path="/4EA1F56E/4EA1E8C1" Ref="R71"  Part="1"
 AR Path="/4EA1D331/4EA1E8C1" Ref="R82"  Part="1"
-F 0 "R71" V 5630 5150 50  0000 C CNN
+F 0 "R82" V 5630 5150 50  0000 C CNN
 F 1 "0R22" V 5550 5150 50  0000 C CNN
 	1    5550 5150
@@
 AR Path="/4EA1F56E/4EA1E8BB" Ref="R72"  Part="1"
 AR Path="/4EA1D331/4EA1E8BB" Ref="R83"  Part="1"
-F 0 "R72" V 5880 5150 50  0000 C CNN
+F 0 "R83" V 5880 5150 50  0000 C CNN
 F 1 "0R22" V 5800 5150 50  0000 C CNN
 	1    5800 5150
@@
 AR Path="/4EA1F56E/4EA1E852" Ref="C56"  Part="1"
 AR Path="/4EA1D331/4EA1E852" Ref="C70"  Part="1"
-F 0 "C56" H 6100 5200 50  0000 L CNN
+F 0 "C70" H 6100 5200 50  0000 L CNN
 F 1 "220nF" H 6100 5000 50  0000 L CNN
 	1    6050 5100
@@
 AR Path="/4EA1F56E/4EA1E80A" Ref="#PWR0116"  Part="1"
 AR Path="/4EA1D331/4EA1E80A" Ref="#PWR0128"  Part="1"
-F 0 "#PWR0116" H 4450 1850 30  0001 C CNN
+F 0 "#PWR0128" H 4450 1850 30  0001 C CNN
 F 1 "GND" H 4450 1780 30  0001 C CNN
 	1    4450 1850
@@
 AR Path="/4EA1F56E/4EA1E7F2" Ref="C47"  Part="1"
 AR Path="/4EA1D331/4EA1E7F2" Ref="C61"  Part="1"
-F 0 "C47" H 4500 1550 50  0000 L CNN
+F 0 "C61" H 4500 1550 50  0000 L CNN
 F 1 "100nF" H 4500 1350 50  0000 L CNN
 	1    4450 1450
@@
 AR Path="/4EA1F56E/4EA1E798" Ref="C49"  Part="1"
 AR Path="/4EA1D331/4EA1E798" Ref="C63"  Part="1"
-F 0 "C49" V 5250 1650 50  0000 L CNN
+F 0 "C63" V 5250 1650 50  0000 L CNN
 F 1 "220nF" V 5250 1300 50  0000 L CNN
 	1    5350 1500
@@
 AR Path="/4EA1F56E/4EA1E774" Ref="C50"  Part="1"
 AR Path="/4EA1D331/4EA1E774" Ref="C64"  Part="1"
-F 0 "C50" H 6100 1600 50  0000 L CNN
+F 0 "C64" H 6100 1600 50  0000 L CNN
 F 1 "220nF" H 6100 1400 50  0000 L CNN
 	1    6050 1500
@@
 AR Path="/4EA1F56E/4EA1E764" Ref="#PWR0117"  Part="1"
 AR Path="/4EA1D331/4EA1E764" Ref="#PWR0129"  Part="1"
-F 0 "#PWR0117" H 5850 950 20  0001 C CNN
+F 0 "#PWR0129" H 5850 950 20  0001 C CNN
 F 1 "+24V" H 5850 1100 30  0000 C CNN
 	1    5850 1000
