File: laserctrl/sd-isp.sch (KiCad schematic (older format))
At the start: 24 parts, among them J1 USB, J2 MICROSD, P2 Exhaust, P3 Assist Air, P4 Chiller, P5 ftdi serial, Q1 BC817, Q2 BC817, Q3 BV807, SW1 Program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

Commit message: Finished rough board space allocation
Parts:
- added C1: 100nF, symbol C
- added R1: 10k, symbol R
Connections:
- wire segments 73 -> 77
Changed lines of the file:
@@
-EESchema Schematic File Version 2  date 2011-11-13T23:13:03 CET
+EESchema Schematic File Version 2  date 2011-11-14T20:41:00 CET
 LIBS:power
 LIBS:device
@@
 Sheet 2 10
 Title ""
-Date "13 nov 2011"
+Date "14 nov 2011"
 Rev ""
 Comp ""
@@
 $EndDescr
 Wire Wire Line
+	2400 4150 2400 4200
+Connection ~ 2800 4750
+Wire Wire Line
+	2950 4750 2400 4750
+Wire Wire Line
 	6050 1450 6050 1300
 Wire Wire Line
@@
 	9300 3200 9200 3200
 Wire Wire Line
-	2950 4750 2800 4750
-Wire Wire Line
 	2800 4750 2800 4800
 Wire Wire Line
@@
 	1250 2050 1250 1800
 Wire Wire Line
-	1550 1800 1200 1800
+	1200 1800 1550 1800
 Connection ~ 3300 2150
 Wire Wire Line
 	3300 2250 3300 1950
 Wire Wire Line
-	3200 2150 3200 2050
+	3200 2050 3200 2150
 Wire Wire Line
 	2450 2050 2450 2150
 Connection ~ 2200 1800
 Wire Wire Line
-	2450 1800 2050 1800
+	2050 1800 2450 1800
 Wire Wire Line
 	2200 1200 2200 1250
@@
 Connection ~ 3200 2150
 Wire Wire Line
-	1200 1950 1550 1950
+	1550 1950 1200 1950
 Wire Wire Line
 	1500 2050 1500 1950
@@
 	1300 3300 1200 3300
 Wire Wire Line
-	1650 4800 1650 4700
+	1650 4700 1650 4800
 Wire Wire Line
 	1650 4150 1650 4200
@@
 	9600 3000 9600 2950
 Wire Wire Line
-	9600 1100 9600 1000
+	9600 1000 9600 1100
 Connection ~ 9600 1050
 Wire Wire Line
-	9600 2450 9600 2550
+	9600 2550 9600 2450
 Wire Wire Line
 	9600 2950 9850 2950
@@
 Wire Wire Line
 	5350 1300 5500 1300
-$Comp
-L GND #PWR016
+Wire Wire Line
+	2800 5400 2400 5400
+Wire Wire Line
+	2400 5400 2400 5300
+Wire Wire Line
+	2400 4900 2400 4700
+Connection ~ 2400 4750
+$Comp
+L +3.3V #PWR016
+U 1 1 4EC159D5
+P 2400 4150
+F 0 "#PWR016" H 2400 4110 30  0001 C CNN
+F 1 "+3.3V" H 2400 4260 30  0000 C CNN
+	1    2400 4150
+	1    0    0    -1
+$EndComp
+$Comp
+L R R1
+U 1 1 4EC1599F
+P 2400 4450
+F 0 "R1" V 2480 4450 50  0000 C CNN
+F 1 "10k" V 2400 4450 50  0000 C CNN
+	1    2400 4450
+	1    0    0    -1
+$EndComp
+$Comp
+L C C1
+U 1 1 4EC1599E
+P 2400 5100
+F 0 "C1" H 2450 5200 50  0000 L CNN
+F 1 "100nF" H 2150 5000 50  0000 L CNN
+	1    2400 5100
+	1    0    0    -1
+$EndComp
+$Comp
+L GND #PWR017
 U 1 1 4EBEC7BB
 P 6050 1450
-F 0 "#PWR016" H 6050 1450 30  0001 C CNN
+F 0 "#PWR017" H 6050 1450 30  0001 C CNN
 F 1 "GND" H 6050 1380 30  0001 C CNN
 	1    6050 1450
@@
 $EndComp
 $Comp
-L +24V #PWR017
+L +24V #PWR018
 U 1 1 4EBAE1E7
 P 9600 2450
-F 0 "#PWR017" H 9600 2400 20  0001 C CNN
+F 0 "#PWR018" H 9600 2400 20  0001 C CNN
 F 1 "+24V" H 9600 2550 30  0000 C CNN
 	1    9600 2450
@@
 $EndComp
 $Comp
-L GND #PWR018
+L GND #PWR019
 U 1 1 4EBAC055
 P 9700 5050
-F 0 "#PWR018" H 9700 5050 30  0001 C CNN
+F 0 "#PWR019" H 9700 5050 30  0001 C CNN
 F 1 "GND" H 9700 4980 30  0001 C CNN
 	1    9700 5050
@@
 $EndComp
 $Comp
-L +3.3V #PWR019
+L +3.3V #PWR020
 U 1 1 4EBAC054
 P 9700 4850
-F 0 "#PWR019" H 9700 4810 30  0001 C CNN
+F 0 "#PWR020" H 9700 4810 30  0001 C CNN
 F 1 "+3.3V" H 9700 4960 30  0000 C CNN
 	1    9700 4850
@@
 RXDC
 $Comp
-L GND #PWR020
+L GND #PWR021
 U 1 1 4EBAC053
 P 8500 5150
-F 0 "#PWR020" H 8500 5150 30  0001 C CNN
+F 0 "#PWR021" H 8500 5150 30  0001 C CNN
 F 1 "GND" H 8500 5080 30  0001 C CNN
 	1    8500 5150
@@
 $EndComp
 $Comp
-L +24V #PWR021
+L +24V #PWR022
 U 1 1 4EBAC052
 P 8500 5400
-F 0 "#PWR021" H 8500 5350 20  0001 C CNN
+F 0 "#PWR022" H 8500 5350 20  0001 C CNN
 F 1 "+24V" H 8500 5500 30  0000 C CNN
 	1    8500 5400
@@
 $EndComp
 $Comp
-L GND #PWR022
+L GND #PWR023
 U 1 1 4EBAC038
 P 9600 2000
-F 0 "#PWR022" H 9600 2000 30  0001 C CNN
+F 0 "#PWR023" H 9600 2000 30  0001 C CNN
 F 1 "GND" H 9600 1930 30  0001 C CNN
 	1    9600 2000
@@
 $EndComp
 $Comp
-L +24V #PWR023
+L +24V #PWR024
 U 1 1 4EBAC035
 P 9600 1000
-F 0 "#PWR023" H 9600 950 20  0001 C CNN
+F 0 "#PWR024" H 9600 950 20  0001 C CNN
 F 1 "+24V" H 9600 1100 30  0000 C CNN
 	1    9600 1000
@@
 $EndComp
 $Comp
-L GND #PWR024
+L GND #PWR025
 U 1 1 4EBAC031
 P 9600 3450
-F 0 "#PWR024" H 9600 3450 30  0001 C CNN
+F 0 "#PWR025" H 9600 3450 30  0001 C CNN
 F 1 "GND" H 9600 3380 30  0001 C CNN
 	1    9600 3450
@@
 $EndComp
 $Comp
-L GND #PWR025
+L GND #PWR026
 U 1 1 4EB6DA7E
 P 1850 6700
-F 0 "#PWR025" H 1850 6700 30  0001 C CNN
+F 0 "#PWR026" H 1850 6700 30  0001 C CNN
 F 1 "GND" H 1850 6630 30  0001 C CNN
 	1    1850 6700
@@
 $EndComp
 $Comp
-L +3.3V #PWR026
+L +3.3V #PWR027
 U 1 1 4EB6DA5E
 P 1850 6400
-F 0 "#PWR026" H 1850 6360 30  0001 C CNN
+F 0 "#PWR027" H 1850 6360 30  0001 C CNN
 F 1 "+3.3V" H 1850 6510 30  0000 C CNN
 	1    1850 6400
@@
 CS
 $Comp
-L GND #PWR027
+L GND #PWR028
 U 1 1 4EB6D76C
 P 2800 5500
-F 0 "#PWR027" H 2800 5500 30  0001 C CNN
+F 0 "#PWR028" H 2800 5500 30  0001 C CNN
 F 1 "GND" H 2800 5430 30  0001 C CNN
 	1    2800 5500
@@
 $EndComp
 $Comp
-L +3.3V #PWR028
+L +3.3V #PWR029
 U 1 1 4EB6D47F
 P 1650 4150
-F 0 "#PWR028" H 1650 4110 30  0001 C CNN
+F 0 "#PWR029" H 1650 4110 30  0001 C CNN
 F 1 "+3.3V" H 1650 4260 30  0000 C CNN
 	1    1650 4150
@@
 $EndComp
 $Comp
-L GND #PWR029
+L GND #PWR030
 U 1 1 4EB6D436
 P 1650 5500
-F 0 "#PWR029" H 1650 5500 30  0001 C CNN
+F 0 "#PWR030" H 1650 5500 30  0001 C CNN
 F 1 "GND" H 1650 5430 30  0001 C CNN
 	1    1650 5500
@@
 $EndComp
 $Comp
-L GND #PWR030
+L GND #PWR031
 U 1 1 4EB6D3CA
 P 1200 3700
-F 0 "#PWR030" H 1200 3700 30  0001 C CNN
+F 0 "#PWR031" H 1200 3700 30  0001 C CNN
 F 1 "GND" H 1200 3630 30  0001 C CNN
 	1    1200 3700
@@
 ~RESET
 $Comp
-L GND #PWR031
+L GND #PWR032
 U 1 1 4EB6D202
 P 1500 2550
-F 0 "#PWR031" H 1500 2550 30  0001 C CNN
+F 0 "#PWR032" H 1500 2550 30  0001 C CNN
 F 1 "GND" H 1500 2480 30  0001 C CNN
 	1    1500 2550
@@
 $EndComp
 $Comp
-L GND #PWR032
+L GND #PWR033
 U 1 1 4EB6D1FB
 P 1250 2550
-F 0 "#PWR032" H 1250 2550 30  0001 C CNN
+F 0 "#PWR033" H 1250 2550 30  0001 C CNN
 F 1 "GND" H 1250 2480 30  0001 C CNN
 	1    1250 2550
@@
 $EndComp
 $Comp
-L GND #PWR033
+L GND #PWR034
 U 1 1 4EB6D1B5
 P 3300 2250
-F 0 "#PWR033" H 3300 2250 30  0001 C CNN
+F 0 "#PWR034" H 3300 2250 30  0001 C CNN
 F 1 "GND" H 3300 2180 30  0001 C CNN
 	1    3300 2250
@@
 $EndComp
 $Comp
-L +3.3V #PWR034
+L +3.3V #PWR035
 U 1 1 4EB6D11C
 P 2200 750
-F 0 "#PWR034" H 2200 710 30  0001 C CNN
+F 0 "#PWR035" H 2200 710 30  0001 C CNN
 F 1 "+3.3V" H 2200 860 30  0000 C CNN
 	1    2200 750
