File: laserctrl/laser.sch (KiCad schematic (older format))
At the start: 36 parts, among them P10 estop, P11 LASER, Q6 BC817, Q7 BC817, Q8 BC817, U2 EL 816S(TA), U3 EL 816S(TA), U4 EL 816S(TA), U5 EL 816S(TA), U6 EL 816S(TA)

Commit message: Use double-shottky diodes in stead of tons of discrete miniMELFs
Parts:
- removed D14: DIODE, symbol DIODE
- added D7, D8, D9: BAT 54S, symbol DIODE2
- D12, D18: value DIODE -> LS 914B
Other:
- moved on the sheet: R27, R32

Commit message: Added a couple of missing modules
Connections:
- wire segments 92 -> 117
Other:
- moved on the sheet: R27
Changed lines of the file:
@@
-EESchema Schematic File Version 2  date 2011-11-09T22:36:32 CET
+EESchema Schematic File Version 2  date 2011-11-10T19:54:24 CET
 LIBS:power
 LIBS:device
@@
 Sheet 4 10
 Title ""
-Date "9 nov 2011"
+Date "10 nov 2011"
 Rev ""
 Comp ""
@@
 	6100 5000 6100 5100
 Wire Wire Line
-	5000 4700 7350 4700
+	5000 4700 6100 4700
+Wire Wire Line
+	6100 4700 6550 4700
+Wire Wire Line
+	6550 4700 7350 4700
 Connection ~ 5700 3900
 Wire Wire Line
-	8150 3900 5000 3900
+	8150 3900 5700 3900
+Wire Wire Line
+	5700 3900 5200 3900
+Wire Wire Line
+	5200 3900 5000 3900
 Connection ~ 5700 3600
 Wire Wire Line
-	6550 3600 5000 3600
-Connection ~ 5200 2650
-Wire Wire Line
-	5000 2650 5600 2650
-Wire Wire Line
-	5000 2950 8150 2950
+	6550 3600 5700 3600
+Wire Wire Line
+	5700 3600 5000 3600
+Connection ~ 5700 2650
+Wire Wire Line
+	5000 2650 5700 2650
+Wire Wire Line
+	5700 2650 5850 2650
+Wire Wire Line
+	5000 2950 5700 2950
+Wire Wire Line
+	5700 2950 7850 2950
+Wire Wire Line
+	7850 2950 8150 2950
 Wire Wire Line
 	5750 1400 6550 1400
 Connection ~ 2800 5700
 Wire Wire Line
-	2650 5700 2950 5700
+	2650 5700 2800 5700
+Wire Wire Line
+	2800 5700 2950 5700
 Wire Wire Line
 	1700 5650 1700 5700
@@
 Connection ~ 1850 3700
 Wire Wire Line
-	1350 2650 3750 2650
+	1350 2650 2800 2650
+Wire Wire Line
+	2800 2650 3600 2650
+Wire Wire Line
+	3600 2650 3750 2650
 Wire Wire Line
 	2900 2000 2800 2000
@@
 	3300 2750 3300 2950
 Wire Wire Line
-	1450 6500 1450 6350
+	1450 6500 1450 6400
+Wire Wire Line
+	1450 6400 1450 6350
 Connection ~ 1450 5900
 Wire Wire Line
@@
 Connection ~ 6550 2650
 Wire Wire Line
-	6100 2650 6550 2650
+	6350 2650 6550 2650
 Connection ~ 5200 3900
 Connection ~ 6550 4700
@@
 	7350 3600 8150 3600
 Wire Wire Line
-	7850 3800 8150 3800
+	7850 3800 8000 3800
+Wire Wire Line
+	8000 3800 8150 3800
 Wire Wire Line
 	3650 3600 3750 3600
@@
 	7850 3700 8150 3700
 Wire Wire Line
-	6550 1400 6550 4100
+	6550 1400 6550 2650
+Wire Wire Line
+	6550 2650 6550 3600
+Wire Wire Line
+	6550 3600 6550 4000
+Wire Wire Line
+	6550 4000 6550 4100
 Connection ~ 6550 4000
 Connection ~ 6550 3600
@@
 	3800 1700 1350 1700
 Wire Wire Line
-	1950 3700 1350 3700
+	1950 3700 1850 3700
+Wire Wire Line
+	1850 3700 1350 3700
 Wire Wire Line
 	1850 3700 1850 3900
@@
 	2950 5000 3750 5000
 Wire Wire Line
-	1950 4800 1350 4800
+	1950 4800 1850 4800
+Wire Wire Line
+	1850 4800 1350 4800
 Wire Wire Line
 	1700 4550 1700 4600
 Wire Wire Line
-	2950 4600 2650 4600
+	2950 4600 2800 4600
+Wire Wire Line
+	2800 4600 2650 4600
 Connection ~ 2800 4600
 Wire Wire Line
-	1350 5900 1950 5900
+	1350 5900 1450 5900
+Wire Wire Line
+	1450 5900 1850 5900
+Wire Wire Line
+	1850 5900 1950 5900
 Connection ~ 5650 1700
 Wire Wire Line
 	5050 1700 5650 1700
 Wire Wire Line
-	5650 1550 5650 1800
+	5650 1550 5650 1700
+Wire Wire Line
+	5650 1700 5650 1800
 Connection ~ 5150 1400
 Wire Wire Line
-	5250 1400 5050 1400
+	5250 1400 5150 1400
+Wire Wire Line
+	5150 1400 5050 1400
 Wire Wire Line
 	5250 1550 5150 1550
@@
 	5150 1550 5150 1400
 Wire Wire Line
-	5200 3350 5200 3250
-Connection ~ 5200 2950
-Wire Wire Line
-	5700 4200 5700 4400
+	5700 3350 5700 3250
+Connection ~ 5700 2950
+Wire Wire Line
+	5700 4200 5700 4250
+Wire Wire Line
+	5700 4250 5700 4400
 Connection ~ 5700 4250
 Connection ~ 6100 4700
@@
 	6100 4400 6100 4000
 Wire Wire Line
-	6100 4000 8150 4000
+	6100 4000 6550 4000
+Wire Wire Line
+	6550 4000 8150 4000
 $Comp
 L GND #PWR042
@@
 L GND #PWR043
 U 1 1 4EBADE5B
-P 5200 3350
-F 0 "#PWR043" H 5200 3350 30  0001 C CNN
-F 1 "GND" H 5200 3280 30  0001 C CNN
-	1    5200 3350
+P 5700 3350
+F 0 "#PWR043" H 5700 3350 30  0001 C CNN
+F 1 "GND" H 5700 3280 30  0001 C CNN
+	1    5700 3350
 	1    0    0    -1
 $EndComp
@@
 L DIODE2 D7
 U 1 1 4EBADE4A
-P 5200 2950
-F 0 "D7" H 5350 3050 60  0000 C CNN
-F 1 "BAT 54S" H 5450 3150 60  0000 C CNN
-	1    5200 2950
+P 5700 2950
+F 0 "D7" H 5850 3050 60  0000 C CNN
+F 1 "BAT 54S" H 5950 3150 60  0000 C CNN
+	1    5700 2950
 	-1   0    0    1
 $EndComp
@@
 L R R27
 U 1 1 4EB1C921
-P 5850 2650
-F 0 "R27" V 5930 2650 50  0000 C CNN
-F 1 "200R" V 5850 2650 50  0000 C CNN
-	1    5850 2650
-	0    1    1    0
-$EndComp
+P 6100 2650
+F 0 "R27" V 6180 2650 50  0000 C CNN
+F 1 "200R" V 6100 2650 50  0000 C CNN
+	1    6100 2650
+	0    1    1    0
+$EndComp

Commit message: Added foot print for a 5V regulator that I can actually get, added 3-way solder jumper, added waterflow sensor input, pinned out the extra pins
Connections:
- wire segments 117 -> 92
Changed lines of the file:
@@
-EESchema Schematic File Version 2  date 2011-11-10T19:54:24 CET
+EESchema Schematic File Version 2  date 2011-11-12T10:43:20 CET
 LIBS:power
 LIBS:device
@@
 LIBS:jumper3
 LIBS:diode2
+LIBS:78l00a
 LIBS:laserctrl-cache
 EELAYER 25  0
@@
 Sheet 4 10
 Title ""
-Date "10 nov 2011"
+Date "12 nov 2011"
 Rev ""
 Comp ""
@@
 	6100 5000 6100 5100
 Wire Wire Line
-	5000 4700 6100 4700
-Wire Wire Line
-	6100 4700 6550 4700
-Wire Wire Line
-	6550 4700 7350 4700
+	5000 4700 7350 4700
 Connection ~ 5700 3900
 Wire Wire Line
-	8150 3900 5700 3900
-Wire Wire Line
-	5700 3900 5200 3900
-Wire Wire Line
-	5200 3900 5000 3900
+	8150 3900 5000 3900
 Connection ~ 5700 3600
 Wire Wire Line
-	6550 3600 5700 3600
-Wire Wire Line
-	5700 3600 5000 3600
+	6550 3600 5000 3600
 Connection ~ 5700 2650
 Wire Wire Line
-	5000 2650 5700 2650
-Wire Wire Line
-	5700 2650 5850 2650
-Wire Wire Line
-	5000 2950 5700 2950
-Wire Wire Line
-	5700 2950 7850 2950
-Wire Wire Line
-	7850 2950 8150 2950
+	5000 2650 5850 2650
+Wire Wire Line
+	5000 2950 8150 2950
 Wire Wire Line
 	5750 1400 6550 1400
 Connection ~ 2800 5700
 Wire Wire Line
-	2650 5700 2800 5700
-Wire Wire Line
-	2800 5700 2950 5700
+	2650 5700 2950 5700
 Wire Wire Line
 	1700 5650 1700 5700
@@
 Connection ~ 1850 3700
 Wire Wire Line
-	1350 2650 2800 2650
-Wire Wire Line
-	2800 2650 3600 2650
-Wire Wire Line
-	3600 2650 3750 2650
+	1350 2650 3750 2650
 Wire Wire Line
 	2900 2000 2800 2000
@@
 	3300 2750 3300 2950
 Wire Wire Line
-	1450 6500 1450 6400
-Wire Wire Line
-	1450 6400 1450 6350
+	1450 6500 1450 6350
 Connection ~ 1450 5900
 Wire Wire Line
@@
 	7350 3600 8150 3600
 Wire Wire Line
-	7850 3800 8000 3800
-Wire Wire Line
-	8000 3800 8150 3800
+	7850 3800 8150 3800
 Wire Wire Line
 	3650 3600 3750 3600
@@
 	7850 3700 8150 3700
 Wire Wire Line
-	6550 1400 6550 2650
-Wire Wire Line
-	6550 2650 6550 3600
-Wire Wire Line
-	6550 3600 6550 4000
-Wire Wire Line
-	6550 4000 6550 4100
+	6550 1400 6550 4100
 Connection ~ 6550 4000
 Connection ~ 6550 3600
@@
 	3800 1700 1350 1700
 Wire Wire Line
-	1950 3700 1850 3700
-Wire Wire Line
-	1850 3700 1350 3700
+	1950 3700 1350 3700
 Wire Wire Line
 	1850 3700 1850 3900
@@
 	2950 5000 3750 5000
 Wire Wire Line
-	1950 4800 1850 4800
-Wire Wire Line
-	1850 4800 1350 4800
+	1950 4800 1350 4800
 Wire Wire Line
 	1700 4550 1700 4600
 Wire Wire Line
-	2950 4600 2800 4600
-Wire Wire Line
-	2800 4600 2650 4600
+	2950 4600 2650 4600
 Connection ~ 2800 4600
 Wire Wire Line
-	1350 5900 1450 5900
-Wire Wire Line
-	1450 5900 1850 5900
-Wire Wire Line
-	1850 5900 1950 5900
+	1350 5900 1950 5900
 Connection ~ 5650 1700
 Wire Wire Line
 	5050 1700 5650 1700
 Wire Wire Line
-	5650 1550 5650 1700
-Wire Wire Line
-	5650 1700 5650 1800
+	5650 1550 5650 1800
 Connection ~ 5150 1400
 Wire Wire Line
-	5250 1400 5150 1400
-Wire Wire Line
-	5150 1400 5050 1400
+	5250 1400 5050 1400
 Wire Wire Line
 	5250 1550 5150 1550
@@
 Connection ~ 5700 2950
 Wire Wire Line
-	5700 4200 5700 4250
-Wire Wire Line
-	5700 4250 5700 4400
+	5700 4200 5700 4400
 Connection ~ 5700 4250
 Connection ~ 6100 4700
@@
 	6100 4400 6100 4000
 Wire Wire Line
-	6100 4000 6550 4000
-Wire Wire Line
-	6550 4000 8150 4000
-$Comp
-L GND #PWR042
+	6100 4000 8150 4000
+$Comp
+L GND #PWR046
 U 1 1 4EBADF3F
 P 6100 5100
-F 0 "#PWR042" H 6100 5100 30  0001 C CNN
+F 0 "#PWR046" H 6100 5100 30  0001 C CNN
 F 1 "GND" H 6100 5030 30  0001 C CNN
 	1    6100 5100
@@
 $EndComp
 $Comp
-L GND #PWR043
+L GND #PWR047
 U 1 1 4EBADE5B
 P 5700 3350
-F 0 "#PWR043" H 5700 3350 30  0001 C CNN
+F 0 "#PWR047" H 5700 3350 30  0001 C CNN
 F 1 "GND" H 5700 3280 30  0001 C CNN
 	1    5700 3350
@@
 $EndComp
 $Comp
-L GND #PWR044
+L GND #PWR048
 U 1 1 4EB44719
 P 2800 6200
-F 0 "#PWR044" H 2800 6200 30  0001 C CNN
+F 0 "#PWR048" H 2800 6200 30  0001 C CNN
 F 1 "GND" H 2800 6130 30  0001 C CNN
 	1    2800 6200
@@
 $EndComp
 $Comp
-L +3.3V #PWR045
+L +3.3V #PWR049
 U 1 1 4EB44715
 P 3100 5750
-F 0 "#PWR045" H 3100 5710 30  0001 C CNN
+F 0 "#PWR049" H 3100 5710 30  0001 C CNN
 F 1 "+3.3V" H 3100 5860 30  0000 C CNN
 	1    3100 5750
@@
 $EndComp
 $Comp
-L +3.3V #PWR046
+L +3.3V #PWR050
 U 1 1 4EB44714
 P 1700 5650
-F 0 "#PWR046" H 1700 5610 30  0001 C CNN
+F 0 "#PWR050" H 1700 5610 30  0001 C CNN
 F 1 "+3.3V" H 1700 5760 30  0000 C CNN
 	1    1700 5650
@@
 $EndComp
 $Comp
-L +3.3V #PWR047
+L +3.3V #PWR051
 U 1 1 4EB44663
 P 1700 4550
-F 0 "#PWR047" H 1700 4510 30  0001 C CNN
+F 0 "#PWR051" H 1700 4510 30  0001 C CNN
 F 1 "+3.3V" H 1700 4660 30  0000 C CNN
 	1    1700 4550
@@
 $EndComp
 $Comp
-L +3.3V #PWR048
+L +3.3V #PWR052
 U 1 1 4EB44559
 P 3100 4650
-F 0 "#PWR048" H 3100 4610 30  0001 C CNN
+F 0 "#PWR052" H 3100 4610 30  0001 C CNN
 F 1 "+3.3V" H 3100 4760 30  0000 C CNN
 	1    3100 4650
@@
 $EndComp
 $Comp
-L GND #PWR049
+L GND #PWR053
 U 1 1 4EB4452F
 P 2800 5100
-F 0 "#PWR049" H 2800 5100 30  0001 C CNN
+F 0 "#PWR053" H 2800 5100 30  0001 C CNN
 F 1 "GND" H 2800 5030 30  0001 C CNN
 	1    2800 5100
@@
 $EndComp
 $Comp
-L +3.3V #PWR050
+L +3.3V #PWR054
 U 1 1 4EB444DA
 P 3100 3550
-F 0 "#PWR050" H 3100 3510 30  0001 C CNN
+F 0 "#PWR054" H 3100 3510 30  0001 C CNN
 F 1 "+3.3V" H 3100 3660 30  0000 C CNN
 	1    3100 3550
@@
 $EndComp
 $Comp
-L GND #PWR051
+L GND #PWR055
 U 1 1 4EB44499
 P 2800 4000
-F 0 "#PWR051" H 2800 4000 30  0001 C CNN
+F 0 "#PWR055" H 2800 4000 30  0001 C CNN
 F 1 "GND" H 2800 3930 30  0001 C CNN
 	1    2800 4000
@@
 $EndComp
 $Comp
-L GND #PWR052
+L GND #PWR056
 U 1 1 4EB43AA5
 P 5650 1800
-F 0 "#PWR052" H 5650 1800 30  0001 C CNN
+F 0 "#PWR056" H 5650 1800 30  0001 C CNN
 F 1 "GND" H 5650 1730 30  0001 C CNN
 	1    5650 1800
@@
 $EndComp
 $Comp
-L GND #PWR053
+L GND #PWR057
 U 1 1 4EB438A1
 P 2800 2100
-F 0 "#PWR053" H 2800 2100 30  0001 C CNN
+F 0 "#PWR057" H 2800 2100 30  0001 C CNN
 F 1 "GND" H 2800 2030 30  0001 C CNN
 	1    2800 2100
@@
 $EndComp
 $Comp
-L +3.3V #PWR054
+L +3.3V #PWR058
 U 1 1 4EB43856
 P 2850 2950
-F 0 "#PWR054" H 2850 2910 30  0001 C CNN
+F 0 "#PWR058" H 2850 2910 30  0001 C CNN
 F 1 "+3.3V" H 2850 3060 30  0000 C CNN
 	1    2850 2950
@@
 $EndComp
 $Comp
-L GND #PWR055
+L GND #PWR059
 U 1 1 4EB1CD19
 P 1450 7150
-F 0 "#PWR055" H 1450 7150 30  0001 C CNN
+F 0 "#PWR059" H 1450 7150 30  0001 C CNN
 F 1 "GND" H 1450 7080 30  0001 C CNN
 	1    1450 7150
@@
 Watchdog ready
 $Comp
-L GND #PWR056
+L GND #PWR060
 U 1 1 4EB1C992
 P 5700 4400
-F 0 "#PWR056" H 5700 4400 30  0001 C CNN
+F 0 "#PWR060" H 5700 4400 30  0001 C CNN
 F 1 "GND" H 5700 4330 30  0001 C CNN
 	1    5700 4400
@@
 $EndComp
 $Comp
-L GND #PWR057
+L GND #PWR061
 U 1 1 4EB1C889
 P 7850 3800
-F 0 "#PWR057" H 7850 3800 30  0001 C CNN
+F 0 "#PWR061" H 7850 3800 30  0001 C CNN
 F 1 "GND" H 7850 3730 30  0001 C CNN
 	1    7850 3800
@@
 $EndComp
 $Comp
-L +3.3V #PWR058
+L +3.3V #PWR062
 U 1 1 4EB1C82C
 P 3650 1300
-F 0 "#PWR058" H 3650 1260 30  0001 C CNN
+F 0 "#PWR062" H 3650 1260 30  0001 C CNN
 F 1 "+3.3V" H 3650 1410 30  0000 C CNN
 	1    3650 1300
@@
 $EndComp
 $Comp
-L GND #PWR059
+L GND #PWR063
 U 1 1 4EB1C714
 P 3600 3050
-F 0 "#PWR059" H 3600 3050 30  0001 C CNN
+F 0 "#PWR063" H 3600 3050 30  0001 C CNN
 F 1 "GND" H 3600 2980 30  0001 C CNN
 	1    3600 3050
@@
 $EndComp
 $Comp
-L +3.3V #PWR060
+L +3.3V #PWR064
 U 1 1 4EB1C6EC
 P 3600 1950
-F 0 "#PWR060" H 3600 1910 30  0001 C CNN
+F 0 "#PWR064" H 3600 1910 30  0001 C CNN
 F 1 "+3.3V" H 3600 2060 30  0000 C CNN
 	1    3600 1950
@@
 $EndComp
 $Comp
-L GND #PWR061
+L GND #PWR065
 U 1 1 4EB1C552
 P 5100 6200
-F 0 "#PWR061" H 5100 6200 30  0001 C CNN
+F 0 "#PWR065" H 5100 6200 30  0001 C CNN
 F 1 "GND" H 5100 6130 30  0001 C CNN
 	1    5100 6200
@@
 LASER Ready
 $Comp
-L GND #PWR062
+L GND #PWR066
 U 1 1 4EAEEABA
 P 8000 2750
-F 0 "#PWR062" H 8000 2750 30  0001 C CNN
+F 0 "#PWR066" H 8000 2750 30  0001 C CNN
 F 1 "GND" H 8000 2680 30  0001 C CNN
 	1    8000 2750

Commit message: Started board space allocation
Parts:
- R25, R28, R34, R38: value 330R -> 150R
Changed lines of the file:
@@
-EESchema Schematic File Version 2  date 2011-11-12T10:43:20 CET
+EESchema Schematic File Version 2  date 2011-11-13T12:04:33 CET
 LIBS:power
 LIBS:device
@@
 LIBS:diode2
 LIBS:78l00a
+LIBS:conn_11x2
 LIBS:laserctrl-cache
 EELAYER 25  0
@@
 Sheet 4 10
 Title ""
-Date "12 nov 2011"
+Date "13 nov 2011"
 Rev ""
 Comp ""
@@
 Comment4 ""
 $EndDescr
+Connection ~ 2800 1700
 Wire Wire Line
 	6100 5000 6100 5100
@@
 	6100 4000 8150 4000
 $Comp
-L GND #PWR046
+L GND #PWR049
 U 1 1 4EBADF3F
 P 6100 5100
-F 0 "#PWR046" H 6100 5100 30  0001 C CNN
+F 0 "#PWR049" H 6100 5100 30  0001 C CNN
 F 1 "GND" H 6100 5030 30  0001 C CNN
 	1    6100 5100
@@
 $EndComp
 $Comp
-L GND #PWR047
+L GND #PWR050
 U 1 1 4EBADE5B
 P 5700 3350
-F 0 "#PWR047" H 5700 3350 30  0001 C CNN
+F 0 "#PWR050" H 5700 3350 30  0001 C CNN
 F 1 "GND" H 5700 3280 30  0001 C CNN
 	1    5700 3350
@@
 P 1950 5700
 F 0 "R38" V 2030 5700 50  0000 C CNN
-F 1 "330R" V 1950 5700 50  0000 C CNN
+F 1 "150R" V 1950 5700 50  0000 C CNN
 	1    1950 5700
 	0    1    1    0
@@
 $EndComp
 $Comp
-L GND #PWR048
+L GND #PWR051
 U 1 1 4EB44719
 P 2800 6200
-F 0 "#PWR048" H 2800 6200 30  0001 C CNN
+F 0 "#PWR051" H 2800 6200 30  0001 C CNN
 F 1 "GND" H 2800 6130 30  0001 C CNN
 	1    2800 6200
@@
 $EndComp
 $Comp
-L +3.3V #PWR049
+L +3.3V #PWR052
 U 1 1 4EB44715
 P 3100 5750
-F 0 "#PWR049" H 3100 5710 30  0001 C CNN
+F 0 "#PWR052" H 3100 5710 30  0001 C CNN
 F 1 "+3.3V" H 3100 5860 30  0000 C CNN
 	1    3100 5750
@@
 $EndComp
 $Comp
-L +3.3V #PWR050
+L +3.3V #PWR053
 U 1 1 4EB44714
 P 1700 5650
-F 0 "#PWR050" H 1700 5610 30  0001 C CNN
+F 0 "#PWR053" H 1700 5610 30  0001 C CNN
 F 1 "+3.3V" H 1700 5760 30  0000 C CNN
 	1    1700 5650
@@
 $EndComp
 $Comp
-L +3.3V #PWR051
+L +3.3V #PWR054
 U 1 1 4EB44663
 P 1700 4550
-F 0 "#PWR051" H 1700 4510 30  0001 C CNN
+F 0 "#PWR054" H 1700 4510 30  0001 C CNN
 F 1 "+3.3V" H 1700 4660 30  0000 C CNN
 	1    1700 4550
@@
 $EndComp
 $Comp
-L +3.3V #PWR052
+L +3.3V #PWR055
 U 1 1 4EB44559
 P 3100 4650
-F 0 "#PWR052" H 3100 4610 30  0001 C CNN
+F 0 "#PWR055" H 3100 4610 30  0001 C CNN
 F 1 "+3.3V" H 3100 4760 30  0000 C CNN
 	1    3100 4650
@@
 $EndComp
 $Comp
-L GND #PWR053
+L GND #PWR056
 U 1 1 4EB4452F
 P 2800 5100
-F 0 "#PWR053" H 2800 5100 30  0001 C CNN
+F 0 "#PWR056" H 2800 5100 30  0001 C CNN
 F 1 "GND" H 2800 5030 30  0001 C CNN
 	1    2800 5100
@@
 $EndComp
 $Comp
-L +3.3V #PWR054
+L +3.3V #PWR057
 U 1 1 4EB444DA
 P 3100 3550
-F 0 "#PWR054" H 3100 3510 30  0001 C CNN
+F 0 "#PWR057" H 3100 3510 30  0001 C CNN
 F 1 "+3.3V" H 3100 3660 30  0000 C CNN
 	1    3100 3550
@@
 $EndComp
 $Comp
-L GND #PWR055
+L GND #PWR058
 U 1 1 4EB44499
 P 2800 4000
-F 0 "#PWR055" H 2800 4000 30  0001 C CNN
+F 0 "#PWR058" H 2800 4000 30  0001 C CNN
 F 1 "GND" H 2800 3930 30  0001 C CNN
 	1    2800 4000
@@
 $EndComp
 $Comp
-L GND #PWR056
+L GND #PWR059
 U 1 1 4EB43AA5
 P 5650 1800
-F 0 "#PWR056" H 5650 1800 30  0001 C CNN
+F 0 "#PWR059" H 5650 1800 30  0001 C CNN
 F 1 "GND" H 5650 1730 30  0001 C CNN
 	1    5650 1800
@@
 $EndComp
 $Comp
-L GND #PWR057
+L GND #PWR060
 U 1 1 4EB438A1
 P 2800 2100
-F 0 "#PWR057" H 2800 2100 30  0001 C CNN
+F 0 "#PWR060" H 2800 2100 30  0001 C CNN
 F 1 "GND" H 2800 2030 30  0001 C CNN
 	1    2800 2100
@@
 P 3050 1800
 F 0 "R25" V 3130 1800 50  0000 C CNN
-F 1 "330R" V 3050 1800 50  0000 C CNN
+F 1 "150R" V 3050 1800 50  0000 C CNN
 	1    3050 1800
 	0    1    1    0
 $EndComp
 $Comp
-L +3.3V #PWR058
+L +3.3V #PWR061
 U 1 1 4EB43856
 P 2850 2950
-F 0 "#PWR058" H 2850 2910 30  0001 C CNN
+F 0 "#PWR061" H 2850 2910 30  0001 C CNN
 F 1 "+3.3V" H 2850 3060 30  0000 C CNN
 	1    2850 2950
@@
 P 3050 2750
 F 0 "R28" V 3130 2750 50  0000 C CNN
-F 1 "330R" V 3050 2750 50  0000 C CNN
+F 1 "150R" V 3050 2750 50  0000 C CNN
 	1    3050 2750
 	0    1    1    0
@@
 $EndComp
 $Comp
-L GND #PWR059
+L GND #PWR062
 U 1 1 4EB1CD19
 P 1450 7150
-F 0 "#PWR059" H 1450 7150 30  0001 C CNN
+F 0 "#PWR062" H 1450 7150 30  0001 C CNN
 F 1 "GND" H 1450 7080 30  0001 C CNN
 	1    1450 7150
@@
 Watchdog ready
 $Comp
-L GND #PWR060
+L GND #PWR063
 U 1 1 4EB1C992
 P 5700 4400
-F 0 "#PWR060" H 5700 4400 30  0001 C CNN
+F 0 "#PWR063" H 5700 4400 30  0001 C CNN
 F 1 "GND" H 5700 4330 30  0001 C CNN
 	1    5700 4400
@@
 $EndComp
 $Comp
-L GND #PWR061
+L GND #PWR064
 U 1 1 4EB1C889
 P 7850 3800
-F 0 "#PWR061" H 7850 3800 30  0001 C CNN
+F 0 "#PWR064" H 7850 3800 30  0001 C CNN
 F 1 "GND" H 7850 3730 30  0001 C CNN
 	1    7850 3800
@@
 $EndComp
 $Comp
-L +3.3V #PWR062
+L +3.3V #PWR065
 U 1 1 4EB1C82C
 P 3650 1300
-F 0 "#PWR062" H 3650 1260 30  0001 C CNN
+F 0 "#PWR065" H 3650 1260 30  0001 C CNN
 F 1 "+3.3V" H 3650 1410 30  0000 C CNN
 	1    3650 1300
@@
 $EndComp
 $Comp
-L GND #PWR063
+L GND #PWR066
 U 1 1 4EB1C714
 P 3600 3050
-F 0 "#PWR063" H 3600 3050 30  0001 C CNN
+F 0 "#PWR066" H 3600 3050 30  0001 C CNN
 F 1 "GND" H 3600 2980 30  0001 C CNN
 	1    3600 3050
@@
 $EndComp
 $Comp
-L +3.3V #PWR064
+L +3.3V #PWR067
 U 1 1 4EB1C6EC
 P 3600 1950
-F 0 "#PWR064" H 3600 1910 30  0001 C CNN
+F 0 "#PWR067" H 3600 1910 30  0001 C CNN
 F 1 "+3.3V" H 3600 2060 30  0000 C CNN
 	1    3600 1950
@@
 $EndComp
 $Comp
-L GND #PWR065
+L GND #PWR068
 U 1 1 4EB1C552
 P 5100 6200
-F 0 "#PWR065" H 5100 6200 30  0001 C CNN
+F 0 "#PWR068" H 5100 6200 30  0001 C CNN
 F 1 "GND" H 5100 6130 30  0001 C CNN
 	1    5100 6200
@@
 P 1950 4600
 F 0 "R34" V 2030 4600 50  0000 C CNN
-F 1 "330R" V 1950 4600 50  0000 C CNN
+F 1 "150R" V 1950 4600 50  0000 C CNN
 	1    1950 4600
 	0    1    1    0
@@
 LASER Ready
 $Comp
-L GND #PWR066
+L GND #PWR069
 U 1 1 4EAEEABA
 P 8000 2750
-F 0 "#PWR066" H 8000 2750 30  0001 C CNN
+F 0 "#PWR069" H 8000 2750 30  0001 C CNN
 F 1 "GND" H 8000 2680 30  0001 C CNN
 	1    8000 2750
