File: laserctrl/temp-sensors.sch (KiCad schematic (older format))
At the start: 27 parts, among them P26 waterflow, P6 t-int, P7 t-in, P8 t-out, P9 airflow, Q4 BC807, Q5 BC807

Commit message: Finished rough board space allocation
Parts:
- removed D31: LED, symbol LED
- removed R93: 330, symbol R
Connections:
- wire segments 57 -> 54
Other:
- moved on the sheet: R94

Commit message: Moved things about a bit
Parts:
- added P1: CONN_1, symbol CONN_1
Connections:
- wire segments 54 -> 55
Changed lines of the file:
@@
-EESchema Schematic File Version 2  date 2011-11-14T20:41:00 CET
+EESchema Schematic File Version 2  date 2011-11-16T00:00:22 CET
 LIBS:power
 LIBS:device
@@
 Sheet 3 10
 Title ""
-Date "14 nov 2011"
+Date "15 nov 2011"
 Rev ""
 Comp ""
@@
 $EndDescr
 Wire Wire Line
-	5500 3900 5100 3900
-Wire Wire Line
-	1300 5000 1300 4700
-Connection ~ 2000 3950
-Wire Wire Line
-	2000 3900 2000 4200
-Wire Wire Line
-	2250 3950 2000 3950
-Wire Wire Line
-	2300 3700 2550 3700
-Wire Wire Line
-	2550 3050 2550 3150
-Wire Wire Line
-	1300 5000 2550 5000
-Connection ~ 1550 4400
-Wire Wire Line
-	1550 4400 1550 4500
-Wire Wire Line
-	1550 4900 1550 5000
-Connection ~ 2550 4400
-Wire Wire Line
-	2550 5100 2550 4800
-Connection ~ 2550 5000
-Connection ~ 1550 5000
-Connection ~ 5250 2400
-Connection ~ 5500 2400
-Wire Wire Line
-	5500 2500 5500 2200
-Connection ~ 5500 1800
-Wire Wire Line
-	5250 2300 5250 2400
-Wire Wire Line
-	5250 1800 5250 1900
-Connection ~ 5250 1800
-Wire Wire Line
-	5500 1700 5500 2000
-Wire Wire Line
-	5500 1100 5500 1200
-Wire Wire Line
-	3700 1100 3700 1200
-Wire Wire Line
-	3700 1700 3700 2000
-Connection ~ 3450 1800
-Wire Wire Line
-	3450 1800 3450 1900
-Wire Wire Line
-	3450 2300 3450 2400
-Connection ~ 3700 1800
-Wire Wire Line
-	3700 2500 3700 2200
-Connection ~ 3700 2400
-Connection ~ 3450 2400
-Connection ~ 1850 2400
-Connection ~ 2100 2400
-Wire Wire Line
-	2100 2500 2100 2200
-Connection ~ 2100 1800
-Wire Wire Line
-	1500 1800 2100 1800
-Wire Wire Line
-	1850 2300 1850 2400
-Wire Wire Line
-	1850 1800 1850 1900
-Connection ~ 1850 1800
-Wire Wire Line
-	2100 1700 2100 2000
-Wire Wire Line
-	2100 1100 2100 1200
-Wire Wire Line
-	2550 4400 2500 4400
-Wire Wire Line
-	1800 4450 1800 4400
-Connection ~ 1800 4400
-Wire Wire Line
-	1800 5000 1800 4950
-Connection ~ 1800 5000
-Wire Wire Line
-	2550 3150 2000 3150
-Wire Wire Line
-	2000 3150 2000 3500
-Wire Wire Line
-	2550 3650 2550 3750
-Connection ~ 2550 3700
-Wire Wire Line
-	2500 4200 2550 4200
-Wire Wire Line
-	2550 4150 2550 4600
-Connection ~ 2550 4200
-Wire Wire Line
-	1600 1500 1600 1100
-Wire Wire Line
-	3200 1500 3200 1100
-Connection ~ 3200 1800
-Wire Wire Line
-	3100 1800 3700 1800
-Wire Wire Line
-	3700 2400 3200 2400
-Wire Wire Line
-	3200 2400 3200 2100
-Wire Wire Line
-	5000 1500 5000 1100
-Connection ~ 5000 1800
-Wire Wire Line
-	4900 1800 5500 1800
-Wire Wire Line
-	5500 2400 5000 2400
-Wire Wire Line
-	5000 2400 5000 2100
-Connection ~ 1300 4400
-Wire Wire Line
-	2000 4400 1200 4400
-Wire Wire Line
-	1300 4100 1300 3700
-Wire Wire Line
-	5750 5000 5750 4800
-Wire Wire Line
-	5500 4300 5500 3850
-Connection ~ 5500 4600
-Wire Wire Line
-	5750 4600 4800 4600
-Connection ~ 5500 5000
-Connection ~ 5500 3900
+	2450 2650 2450 2550
+Connection ~ 1600 1800
+Wire Wire Line
+	1600 2100 1600 2400
+Wire Wire Line
+	1600 2400 2100 2400
+Wire Wire Line
+	5500 4900 5500 5100
+Wire Wire Line
+	5100 5000 5750 5000
+Wire Wire Line
+	5100 4000 5100 3900
 Connection ~ 5100 4600
 Wire Wire Line
 	5100 4600 5100 4500
 Connection ~ 5100 4600
-Wire Wire Line
-	5100 3900 5100 4000
-Wire Wire Line
-	5100 5000 5750 5000
-Wire Wire Line
-	5500 4900 5500 5100
-Wire Wire Line
-	2100 2400 1600 2400
-Wire Wire Line
-	1600 2400 1600 2100
-Connection ~ 1600 1800
+Connection ~ 5500 3900
+Connection ~ 5500 5000
+Wire Wire Line
+	5750 4600 4800 4600
+Connection ~ 5500 4600
+Wire Wire Line
+	5500 4300 5500 3850
+Wire Wire Line
+	5750 5000 5750 4800
+Wire Wire Line
+	1300 4100 1300 3700
+Wire Wire Line
+	2000 4400 1200 4400
+Connection ~ 1300 4400
+Wire Wire Line
+	5000 2100 5000 2400
+Wire Wire Line
+	5000 2400 5500 2400
+Wire Wire Line
+	4900 1800 5500 1800
+Connection ~ 5000 1800
+Wire Wire Line
+	5000 1500 5000 1100
+Wire Wire Line
+	3200 2100 3200 2400
+Wire Wire Line
+	3200 2400 3700 2400
+Wire Wire Line
+	3100 1800 3700 1800
+Connection ~ 3200 1800
+Wire Wire Line
+	3200 1500 3200 1100
+Wire Wire Line
+	1600 1500 1600 1100
+Connection ~ 2550 4200
+Wire Wire Line
+	2550 4150 2550 4600
+Wire Wire Line
+	2500 4200 2550 4200
+Connection ~ 2550 3700
+Wire Wire Line
+	2550 3650 2550 3750
+Wire Wire Line
+	2000 3500 2000 3150
+Wire Wire Line
+	2000 3150 2550 3150
+Connection ~ 1800 5000
+Wire Wire Line
+	1800 5000 1800 4950
+Connection ~ 1800 4400
+Wire Wire Line
+	1800 4450 1800 4400
+Wire Wire Line
+	2550 4400 2500 4400
+Wire Wire Line
+	2100 1100 2100 1200
+Wire Wire Line
+	2100 1700 2100 2000
+Connection ~ 1850 1800
+Wire Wire Line
+	1850 1800 1850 1900
+Wire Wire Line
+	1850 2300 1850 2400
+Wire Wire Line
+	1500 1800 2100 1800
+Connection ~ 2100 1800
+Wire Wire Line
+	2100 2500 2100 2200
+Connection ~ 2100 2400
+Connection ~ 1850 2400
+Connection ~ 3450 2400
+Connection ~ 3700 2400
+Wire Wire Line
+	3700 2500 3700 2200
+Connection ~ 3700 1800
+Wire Wire Line
+	3450 2300 3450 2400
+Wire Wire Line
+	3450 1800 3450 1900
+Connection ~ 3450 1800
+Wire Wire Line
+	3700 1700 3700 2000
+Wire Wire Line
+	3700 1100 3700 1200
+Wire Wire Line
+	5500 1100 5500 1200
+Wire Wire Line
+	5500 1700 5500 2000
+Connection ~ 5250 1800
+Wire Wire Line
+	5250 1800 5250 1900
+Wire Wire Line
+	5250 2300 5250 2400
+Connection ~ 5500 1800
+Wire Wire Line
+	5500 2500 5500 2200
+Connection ~ 5500 2400
+Connection ~ 5250 2400
+Connection ~ 1550 5000
+Connection ~ 2550 5000
+Wire Wire Line
+	2550 5100 2550 4800
+Connection ~ 2550 4400
+Wire Wire Line
+	1550 4900 1550 5000
+Wire Wire Line
+	1550 4400 1550 4500
+Connection ~ 1550 4400
+Wire Wire Line
+	2550 5000 1300 5000
+Wire Wire Line
+	2550 3150 2550 3050
+Wire Wire Line
+	2300 3700 2550 3700
+Wire Wire Line
+	2250 3950 2000 3950
+Wire Wire Line
+	2000 3900 2000 4200
+Connection ~ 2000 3950
+Wire Wire Line
+	1300 5000 1300 4700
+Wire Wire Line
+	5100 3900 5500 3900
+$Comp
+L GND #PWR036
+U 1 1 4EC2E64F
+P 2450 2650
+F 0 "#PWR036" H 2450 2650 30  0001 C CNN
+F 1 "GND" H 2450 2580 30  0001 C CNN
+	1    2450 2650
+	1    0    0    -1
+$EndComp
+$Comp
+L CONN_1 P1
+U 1 1 4EC2E647
+P 2450 2400
+F 0 "P1" H 2530 2400 40  0000 L CNN
+F 1 "CONN_1" H 2450 2455 30  0001 C CNN
+	1    2450 2400
+	0    -1   -1   0
+$EndComp
 $Comp
 L DIODE2 D3
@@
 $EndComp
 $Comp
-L +3.3VADC #PWR036
+L +3.3VADC #PWR037
 U 1 1 4EB52427
 P 1600 1100
-F 0 "#PWR036" H 1600 1220 20  0001 C CNN
+F 0 "#PWR037" H 1600 1220 20  0001 C CNN
 F 1 "+3.3VADC" H 1600 1190 30  0000 C CNN
 	1    1600 1100
@@
 $EndComp
 $Comp
-L +3.3V #PWR037
+L +3.3V #PWR038
 U 1 1 4EBE3D7B
 P 5500 3850
-F 0 "#PWR037" H 5500 3810 30  0001 C CNN
+F 0 "#PWR038" H 5500 3810 30  0001 C CNN
 F 1 "+3.3V" H 5500 3960 30  0000 C CNN
 	1    5500 3850
@@
 $EndComp
 $Comp
-L GND #PWR038
+L GND #PWR039
 U 1 1 4EBE3D77
 P 5500 5100
-F 0 "#PWR038" H 5500 5100 30  0001 C CNN
+F 0 "#PWR039" H 5500 5100 30  0001 C CNN
 F 1 "GND" H 5500 5030 30  0001 C CNN
 	1    5500 5100
@@
 $EndComp
 $Comp
-L +3.3VADC #PWR039
+L +3.3VADC #PWR040
 U 1 1 4EBAE2EF
 P 5000 1100
-F 0 "#PWR039" H 5000 1220 20  0001 C CNN
+F 0 "#PWR040" H 5000 1220 20  0001 C CNN
 F 1 "+3.3VADC" H 5000 1190 30  0000 C CNN
 	1    5000 1100
@@
 $EndComp
 $Comp
-L +3.3VADC #PWR040
+L +3.3VADC #PWR041
 U 1 1 4EBAE2E3
 P 3200 1100
-F 0 "#PWR040" H 3200 1220 20  0001 C CNN
+F 0 "#PWR041" H 3200 1220 20  0001 C CNN
 F 1 "+3.3VADC" H 3200 1190 30  0000 C CNN
 	1    3200 1100
@@
 10mA\nconstant current
 $Comp
-L +24V #PWR041
+L +24V #PWR042
 U 1 1 4EB542F9
 P 2550 3050
-F 0 "#PWR041" H 2550 3000 20  0001 C CNN
+F 0 "#PWR042" H 2550 3000 20  0001 C CNN
 F 1 "+24V" H 2550 3150 30  0000 C CNN
 	1    2550 3050
@@
 $EndComp
 $Comp
-L AGND #PWR042
+L AGND #PWR043
 U 1 1 4EB5260B
 P 2550 5100
-F 0 "#PWR042" H 2550 5100 40  0001 C CNN
+F 0 "#PWR043" H 2550 5100 40  0001 C CNN
 F 1 "AGND" H 2550 5030 50  0000 C CNN
 	1    2550 5100
@@
 $EndComp
 $Comp
-L +3.3VADC #PWR043
+L +3.3VADC #PWR044
 U 1 1 4EB52606
 P 1300 3700
-F 0 "#PWR043" H 1300 3820 20  0001 C CNN
+F 0 "#PWR044" H 1300 3820 20  0001 C CNN
 F 1 "+3.3VADC" H 1300 3790 30  0000 C CNN
 	1    1300 3700
@@
 $EndComp
 $Comp
-L +5V #PWR044
+L +5V #PWR045
 U 1 1 4EB52596
 P 5500 1100
-F 0 "#PWR044" H 5500 1190 20  0001 C CNN
+F 0 "#PWR045" H 5500 1190 20  0001 C CNN
 F 1 "+5V" H 5500 1190 30  0000 C CNN
 	1    5500 1100
@@
 laser-out
 $Comp
-L AGND #PWR045
+L AGND #PWR046
 U 1 1 4EB52594
 P 5500 2500
-F 0 "#PWR045" H 5500 2500 40  0001 C CNN
+F 0 "#PWR046" H 5500 2500 40  0001 C CNN
 F 1 "AGND" H 5500 2430 50  0000 C CNN
 	1    5500 2500
@@
 $EndComp
 $Comp
-L AGND #PWR046
+L AGND #PWR047
 U 1 1 4EB5253E
 P 3700 2500
-F 0 "#PWR046" H 3700 2500 40  0001 C CNN
+F 0 "#PWR047" H 3700 2500 40  0001 C CNN
 F 1 "AGND" H 3700 2430 50  0000 C CNN
 	1    3700 2500
@@
 $EndComp
 $Comp
-L +5V #PWR047
+L +5V #PWR048
 U 1 1 4EB5253C
 P 3700 1100
-F 0 "#PWR047" H 3700 1190 20  0001 C CNN
+F 0 "#PWR048" H 3700 1190 20  0001 C CNN
 F 1 "+5V" H 3700 1190 30  0000 C CNN
 	1    3700 1100
@@
 $EndComp
 $Comp
-L +5V #PWR048
+L +5V #PWR049
 U 1 1 4EB523C5
 P 2100 1100
-F 0 "#PWR048" H 2100 1190 20  0001 C CNN
+F 0 "#PWR049" H 2100 1190 20  0001 C CNN
 F 1 "+5V" H 2100 1190 30  0000 C CNN
 	1    2100 1100
@@
 Internal
 $Comp
-L AGND #PWR049
+L AGND #PWR050
 U 1 1 4EB472F1
 P 2100 2500
-F 0 "#PWR049" H 2100 2500 40  0001 C CNN
+F 0 "#PWR050" H 2100 2500 40  0001 C CNN
 F 1 "AGND" H 2100 2430 50  0000 C CNN
 	1    2100 2500
