File: laserctrl/temp-sensors.sch (KiCad schematic (older format))
At the start: 26 parts, among them P1 CONN_1, P26 waterflow, P6 t-int, P7 t-in, P8 t-out, P9 airflow, Q4 BC807, Q5 BC807

Commit message: Checked footprints and fixed 1 thinko on the ARM and unfucked the transistor foot prints
Parts:
- removed Q4, Q5: BC807, symbol PNP
- added Q4, Q5: BC807, symbol BC807
Changed lines of the file:
@@
-EESchema Schematic File Version 2  date 2011-12-03T21:12:32 CET
+EESchema Schematic File Version 2  date 2011-12-07T22:22:26 CET
 LIBS:power
 LIBS:device
@@
 LIBS:78l00a
 LIBS:conn_11x2
+LIBS:bc807
+LIBS:bc817
 LIBS:laserctrl-cache
 EELAYER 25  0
@@
 Sheet 3 10
 Title ""
-Date "3 dec 2011"
+Date "7 dec 2011"
 Rev ""
 Comp ""
@@
 Comment4 ""
 $EndDescr
+$Comp
+L BC807 Q5
+U 1 1 4EDFC6E6
+P 2450 3950
+F 0 "Q5" H 2750 3850 60  0000 R CNN
+F 1 "BC807" H 2950 3950 60  0000 R CNN
+	1    2450 3950
+	1    0    0    1
+$EndComp
+$Comp
+L BC807 Q4
+U 1 1 4EDFC6E1
+P 2100 3700
+F 0 "Q4" H 2100 3550 60  0000 R CNN
+F 1 "BC807" H 2550 3650 60  0000 R CNN
+	1    2100 3700
+	-1   0    0    1
+$EndComp
 Wire Wire Line
 	2450 2650 2450 2550
@@
 $EndComp
 $Comp
-L PNP Q4
-U 1 1 4EB542BA
-P 2100 3700
-F 0 "Q4" H 2100 3550 60  0000 R CNN
-F 1 "BC807" V 2350 3700 60  0000 R CNN
-	1    2100 3700
-	-1   0    0    1
-$EndComp
-$Comp
-L PNP Q5
-U 1 1 4EB542A8
-P 2450 3950
-F 0 "Q5" H 2450 3800 60  0000 R CNN
-F 1 "BC807" H 2950 3900 60  0000 R CNN
-	1    2450 3950
-	1    0    0    1
-$EndComp
-$Comp

Commit message: Started redoing the PCB
Parts:
- P1: value CONN_1 -> 2mm-hole
Changed lines of the file:
@@
-EESchema Schematic File Version 2  date Sun 14 Oct 2012 09:24:14 PM CEST
+EESchema Schematic File Version 2  date Mon 15 Oct 2012 07:59:43 PM CEST
 LIBS:power
 LIBS:device
@@
 LIBS:vo-2630
 LIBS:little-logic
+LIBS:con-molex
+LIBS:con-molex-2
 LIBS:laserctrl-cache
 EELAYER 25  0
@@
 Sheet 4 11
 Title ""
-Date "14 oct 2012"
+Date "15 oct 2012"
 Rev ""
 Comp ""
@@
 	5100 3900 5500 3900
 $Comp
-L GND #PWR037
+L GND #PWR041
 U 1 1 4EC2E64F
 P 2450 2650
-F 0 "#PWR037" H 2450 2650 30  0001 C CNN
+F 0 "#PWR041" H 2450 2650 30  0001 C CNN
 F 1 "GND" H 2450 2580 30  0001 C CNN
 	1    2450 2650
@@
 P 2450 2400
 F 0 "P1" H 2530 2400 40  0000 L CNN
-F 1 "CONN_1" H 2450 2455 30  0001 C CNN
+F 1 "2mm-hole" H 2450 2455 30  0001 C CNN
 	1    2450 2400
 	0    -1   -1   0
@@
 $EndComp
 $Comp
-L +3.3VADC #PWR038
+L +3.3VADC #PWR042
 U 1 1 4EB52427
 P 1600 1100
-F 0 "#PWR038" H 1600 1220 20  0001 C CNN
+F 0 "#PWR042" H 1600 1220 20  0001 C CNN
 F 1 "+3.3VADC" H 1600 1190 30  0000 C CNN
 	1    1600 1100
@@
 $EndComp
 $Comp
-L +3.3V #PWR039
+L +3.3V #PWR043
 U 1 1 4EBE3D7B
 P 5500 3850
-F 0 "#PWR039" H 5500 3810 30  0001 C CNN
+F 0 "#PWR043" H 5500 3810 30  0001 C CNN
 F 1 "+3.3V" H 5500 3960 30  0000 C CNN
 	1    5500 3850
@@
 $EndComp
 $Comp
-L GND #PWR040
+L GND #PWR044
 U 1 1 4EBE3D77
 P 5500 5100
-F 0 "#PWR040" H 5500 5100 30  0001 C CNN
+F 0 "#PWR044" H 5500 5100 30  0001 C CNN
 F 1 "GND" H 5500 5030 30  0001 C CNN
 	1    5500 5100
@@
 $EndComp
 $Comp
-L +3.3VADC #PWR041
+L +3.3VADC #PWR045
 U 1 1 4EBAE2EF
 P 5000 1100
-F 0 "#PWR041" H 5000 1220 20  0001 C CNN
+F 0 "#PWR045" H 5000 1220 20  0001 C CNN
 F 1 "+3.3VADC" H 5000 1190 30  0000 C CNN
 	1    5000 1100
@@
 $EndComp
 $Comp
-L +3.3VADC #PWR042
+L +3.3VADC #PWR046
 U 1 1 4EBAE2E3
 P 3200 1100
-F 0 "#PWR042" H 3200 1220 20  0001 C CNN
+F 0 "#PWR046" H 3200 1220 20  0001 C CNN
 F 1 "+3.3VADC" H 3200 1190 30  0000 C CNN
 	1    3200 1100
@@
 10mA\nconstant current
 $Comp
-L +24V #PWR043
+L +24V #PWR047
 U 1 1 4EB542F9
 P 2550 3050
-F 0 "#PWR043" H 2550 3000 20  0001 C CNN
+F 0 "#PWR047" H 2550 3000 20  0001 C CNN
 F 1 "+24V" H 2550 3150 30  0000 C CNN
 	1    2550 3050
@@
 $EndComp
 $Comp
-L AGND #PWR044
+L AGND #PWR048
 U 1 1 4EB5260B
 P 2550 5100
-F 0 "#PWR044" H 2550 5100 40  0001 C CNN
+F 0 "#PWR048" H 2550 5100 40  0001 C CNN
 F 1 "AGND" H 2550 5030 50  0000 C CNN
 	1    2550 5100
@@
 $EndComp
 $Comp
-L +3.3VADC #PWR045
+L +3.3VADC #PWR049
 U 1 1 4EB52606
 P 1300 3700
-F 0 "#PWR045" H 1300 3820 20  0001 C CNN
+F 0 "#PWR049" H 1300 3820 20  0001 C CNN
 F 1 "+3.3VADC" H 1300 3790 30  0000 C CNN
 	1    1300 3700
@@
 $EndComp
 $Comp
-L +5V #PWR046
+L +5V #PWR050
 U 1 1 4EB52596
 P 5500 1100
-F 0 "#PWR046" H 5500 1190 20  0001 C CNN
+F 0 "#PWR050" H 5500 1190 20  0001 C CNN
 F 1 "+5V" H 5500 1190 30  0000 C CNN
 	1    5500 1100
@@
 laser-out
 $Comp
-L AGND #PWR047
+L AGND #PWR051
 U 1 1 4EB52594
 P 5500 2500
-F 0 "#PWR047" H 5500 2500 40  0001 C CNN
+F 0 "#PWR051" H 5500 2500 40  0001 C CNN
 F 1 "AGND" H 5500 2430 50  0000 C CNN
 	1    5500 2500
@@
 $EndComp
 $Comp
-L AGND #PWR048
+L AGND #PWR052
 U 1 1 4EB5253E
 P 3700 2500
-F 0 "#PWR048" H 3700 2500 40  0001 C CNN
+F 0 "#PWR052" H 3700 2500 40  0001 C CNN
 F 1 "AGND" H 3700 2430 50  0000 C CNN
 	1    3700 2500
@@
 $EndComp
 $Comp
-L +5V #PWR049
+L +5V #PWR053
 U 1 1 4EB5253C
 P 3700 1100
-F 0 "#PWR049" H 3700 1190 20  0001 C CNN
+F 0 "#PWR053" H 3700 1190 20  0001 C CNN
 F 1 "+5V" H 3700 1190 30  0000 C CNN
 	1    3700 1100
@@
 $EndComp
 $Comp
-L +5V #PWR050
+L +5V #PWR054
 U 1 1 4EB523C5
 P 2100 1100
-F 0 "#PWR050" H 2100 1190 20  0001 C CNN
+F 0 "#PWR054" H 2100 1190 20  0001 C CNN
 F 1 "+5V" H 2100 1190 30  0000 C CNN
 	1    2100 1100
@@
 Internal
 $Comp
-L AGND #PWR051
+L AGND #PWR055
 U 1 1 4EB472F1
 P 2100 2500
-F 0 "#PWR051" H 2100 2500 40  0001 C CNN
+F 0 "#PWR055" H 2100 2500 40  0001 C CNN
 F 1 "AGND" H 2100 2430 50  0000 C CNN
 	1    2100 2500
