File: laserctrl/auxio.sch (KiCad schematic (older format))
At the start: 1 part, among them P2 auxio

Commit message: Opened laserctrl using 0.201507230931+5980~23~ubuntu14.10.1 and ordered a PCB from Dirty PCB
Changed lines of the file:
@@
-EESchema Schematic File Version 2  date Sat 16 Feb 2013 05:10:34 PM CET
+EESchema Schematic File Version 2
+LIBS:laserctrl-rescue
 LIBS:power
 LIBS:device
@@
 LIBS:memory
 LIBS:xilinx
-LIBS:special
 LIBS:microcontrollers
 LIBS:dsp
@@
 LIBS:1g08
 LIBS:laserctrl-cache
-EELAYER 25  0
+EELAYER 25 0
 EELAYER END
-$Descr A4 11700 8267
+$Descr A4 11693 8268
 encoding utf-8
 Sheet 2 11
@@
 Comment4 ""
 $EndDescr
-Text Notes 2200 2300 0    50   ~ 0
+Text Notes 2200 2500 0    50   ~ 0
 This is part of the 40 pin IO header that connects to\nthe bulkhead breakout board.\n\nNotice that these GPIO pins are unprotected and need proper protection\ncircuitry if they are needed further out.
 Wire Wire Line
@@
 	3600 1900 3750 1900
 $Comp
-L GND #PWR016
+L GND-RESCUE-laserctrl #PWR016
 U 1 1 507B0CE5
 P 3700 2000
+AR Path="/507B0CE5" Ref="#PWR016"  Part="1"
+AR Path="/507B0AFA/507B0CE5" Ref="#PWR016"  Part="1"
 F 0 "#PWR016" H 3700 2000 30  0001 C CNN
 F 1 "GND" H 3700 1930 30  0001 C CNN
+F 2 "" H 3700 2000 60  0001 C CNN
+F 3 "" H 3700 2000 60  0001 C CNN
 	1    3700 2000
 	0    -1   -1   0
@@
 F 0 "#PWR017" H 3700 1450 20  0001 C CNN
 F 1 "+24V" H 3700 1600 30  0000 C CNN
+F 2 "" H 3700 1500 60  0001 C CNN
+F 3 "" H 3700 1500 60  0001 C CNN
 	1    3700 1500
 	0    1    1    0
 $EndComp
 $Comp
-L GND #PWR018
+L GND-RESCUE-laserctrl #PWR018
 U 1 1 507B0BE0
 P 2700 1500
+AR Path="/507B0BE0" Ref="#PWR018"  Part="1"
+AR Path="/507B0AFA/507B0BE0" Ref="#PWR018"  Part="1"
 F 0 "#PWR018" H 2700 1500 30  0001 C CNN
 F 1 "GND" H 2700 1430 30  0001 C CNN
+F 2 "" H 2700 1500 60  0001 C CNN
+F 3 "" H 2700 1500 60  0001 C CNN
 	1    2700 1500
 	0    1    1    0
@@
 F 0 "#PWR019" H 3850 1520 20  0001 C CNN
 F 1 "+3.3VADC" H 3850 1490 30  0000 C CNN
+F 2 "" H 3850 1400 60  0001 C CNN
+F 3 "" H 3850 1400 60  0001 C CNN
 	1    3850 1400
 	0    1    1    0
@@
 F 0 "#PWR020" H 2600 1400 40  0001 C CNN
 F 1 "AGND" H 2600 1330 50  0000 C CNN
+F 2 "" H 2600 1400 60  0001 C CNN
+F 3 "" H 2600 1400 60  0001 C CNN
 	1    2600 1400
 	0    1    1    0
 $EndComp
 $Comp
-L +3.3V #PWR021
+L +3.3V-RESCUE-laserctrl #PWR021
 U 1 1 507B0BA0
 P 3700 1300
+AR Path="/507B0BA0" Ref="#PWR021"  Part="1"
+AR Path="/507B0AFA/507B0BA0" Ref="#PWR021"  Part="1"
 F 0 "#PWR021" H 3700 1260 30  0001 C CNN
 F 1 "+3.3V" H 3700 1410 30  0000 C CNN
+F 2 "" H 3700 1300 60  0001 C CNN
+F 3 "" H 3700 1300 60  0001 C CNN
 	1    3700 1300
 	0    1    1    0
 $EndComp
 $Comp
-L GND #PWR022
+L GND-RESCUE-laserctrl #PWR022
 U 1 1 507B0B88
 P 2700 1300
+AR Path="/507B0B88" Ref="#PWR022"  Part="1"
+AR Path="/507B0AFA/507B0B88" Ref="#PWR022"  Part="1"
 F 0 "#PWR022" H 2700 1300 30  0001 C CNN
 F 1 "GND" H 2700 1230 30  0001 C CNN
+F 2 "" H 2700 1300 60  0001 C CNN
+F 3 "" H 2700 1300 60  0001 C CNN
 	1    2700 1300
 	0    1    1    0
@@
 F 0 "P2" H 3200 2100 60  0000 C CNN
 F 1 "auxio" V 3200 1650 50  0000 C CNN
+F 2 "" H 3200 1650 60  0001 C CNN
+F 3 "" H 3200 1650 60  0001 C CNN
 	1    3200 1650
 	1    0    0    -1

Commit message: Added aiming shutter
Parts:
- P2: symbol CONN_8X2 -> 1g08:CONN_8X2
Changed lines of the file:
@@
-EESchema Schematic File Version 2
-LIBS:laserctrl-rescue
-LIBS:power
-LIBS:device
-LIBS:transistors
-LIBS:conn
-LIBS:linear
-LIBS:regul
-LIBS:74xx
-LIBS:cmos4000
-LIBS:adc-dac
-LIBS:memory
-LIBS:xilinx
-LIBS:microcontrollers
-LIBS:dsp
-LIBS:microchip
-LIBS:analog_switches
-LIBS:motorola
-LIBS:texas
-LIBS:intel
-LIBS:audio
-LIBS:interface
-LIBS:digital-audio
-LIBS:philips
-LIBS:display
-LIBS:cypress
-LIBS:siliconi
-LIBS:opto
-LIBS:contrib
-LIBS:valves
-LIBS:mounting
-LIBS:23k256
-LIBS:tps78233
-LIBS:drv8811
-LIBS:mcu-nxp
-LIBS:opto-transistor-4p2
-LIBS:atmega328p-a
-LIBS:atmel
-LIBS:microsd
-LIBS:jumper3
-LIBS:diode2
-LIBS:78l00a
-LIBS:conn_11x2
-LIBS:bc807
-LIBS:bc817
-LIBS:vo-2630
-LIBS:little-logic
-LIBS:con-molex
-LIBS:con-molex-2
-LIBS:1g08
+EESchema Schematic File Version 4
 LIBS:laserctrl-cache
-EELAYER 25 0
+EELAYER 26 0
 EELAYER END
 $Descr A4 11693 8268
@@
 	3600 1900 3750 1900
 $Comp
-L GND-RESCUE-laserctrl #PWR016
+L laserctrl-rescue:GND-RESCUE-laserctrl #PWR016
 U 1 1 507B0CE5
 P 3700 2000
@@
 aux0
 $Comp
-L +24V #PWR017
+L power:+24V #PWR017
 U 1 1 507B0BE8
 P 3700 1500
@@
 $EndComp
 $Comp
-L GND-RESCUE-laserctrl #PWR018
+L laserctrl-rescue:GND-RESCUE-laserctrl #PWR018
 U 1 1 507B0BE0
 P 2700 1500
@@
 $EndComp
 $Comp
-L +3.3VADC #PWR019
+L power:+3.3VADC #PWR019
 U 1 1 507B0BCB
 P 3850 1400
@@
 $EndComp
 $Comp
-L AGND #PWR020
+L 1g08:AGND #PWR020
 U 1 1 507B0BAC
 P 2600 1400
@@
 $EndComp
 $Comp
-L +3.3V-RESCUE-laserctrl #PWR021
+L laserctrl-rescue:+3.3V-RESCUE-laserctrl #PWR021
 U 1 1 507B0BA0
 P 3700 1300
@@
 $EndComp
 $Comp
-L GND-RESCUE-laserctrl #PWR022
+L laserctrl-rescue:GND-RESCUE-laserctrl #PWR022
 U 1 1 507B0B88
 P 2700 1300
@@
 $EndComp
 $Comp
-L CONN_8X2 P2
+L 1g08:CONN_8X2 P2
 U 1 1 507B0B80
 P 3200 1650
